Commit message: elbow_flex and shoulder_out: slider zero is now the rest pose
Simon: the elbow slider bends the arm DOWN. Both elbows ran entirely NEGATIVE
(-1.396 .. -0.262) with home at the TOP of that range, so from rest the slider could only
travel one way and that way felt backwards.

Both are now [0, span] with home 0 — slider zero is the straight arm, positive flexes it.
The physical motion is unchanged: invert flips to compensate, so the servo still runs
5 -> 90 as the arm bends.

shoulder_out had the same shape of bug and was arguably worse, though nobody reported it.
Its range was [0.087, 1.047], so ZERO WAS OUTSIDE THE LIMITS —
joint_state_publisher_gui only starts a slider at zero when zero is in range, otherwise it
starts at the MIDPOINT. Launching against real hardware therefore commanded both shoulders
to mid-travel immediately: an unrequested arm movement at start-up. Also re-based to
[0, 0.960] with home 0.

Every driven joint now has its rest pose at slider zero, so a fresh launch commands nothing.

The elbow test encoded the old negative convention. It now asserts the re-based numbers,
EXPECT_FALSE(invert), and that urdf_home_rad is 0 — and its comment no longer claims the
range never contains zero, which stopped being true.

Co-Authored-By: Claude Opus 5 (1M context) <noreply@anthropic.com>
Claude-Session: https://claude.ai/code/session_01Kpk5vJ7u2Qct1dnDk8Kg4X

File: inmoov_description/urdf/config.joints.urdf.xacro (robot description, xacro)
@@ -32,6 +32,6 @@
   <xacro:property name="l_thumb_joint_upper"             value="${r*c['joints']['l_thumb_joint']['maxGoal']}" />
   <xacro:property name="l_thumb_joint_velocity"          value="${r*c['joints']['l_thumb_joint']['maxSpeed']}" />
-  <xacro:property name="l_elbow_flex_joint_lower"        value="${r*c['joints']['l_elbow_flex_joint']['maxGoal']}" />
-  <xacro:property name="l_elbow_flex_joint_upper"        value="${r*c['joints']['l_elbow_flex_joint']['minGoal']}" />
+  <xacro:property name="l_elbow_flex_joint_lower"        value="0" />
+  <xacro:property name="l_elbow_flex_joint_upper"        value="${r*(c['joints']['l_elbow_flex_joint']['minGoal'] - c['joints']['l_elbow_flex_joint']['maxGoal'])}" />
   <xacro:property name="l_elbow_flex_joint_velocity"     value="${r*c['joints']['l_elbow_flex_joint']['maxSpeed']}" />
   <xacro:property name="jaw_joint_lower"                 value="${r*c['joints']['jaw_joint']['minGoal']}" />
@@ -41,6 +41,6 @@
   <xacro:property name="l_wrist_roll_joint_upper"        value="${-(r*(c['joints']['l_wrist_roll_joint']['maxGoal'] - c['joints']['l_wrist_roll_joint']['minGoal'])/2)}" />
   <xacro:property name="l_wrist_roll_joint_velocity"     value="${r*c['joints']['l_wrist_roll_joint']['maxSpeed']}" />
-  <xacro:property name="r_elbow_flex_joint_lower"        value="${r*c['joints']['r_elbow_flex_joint']['maxGoal']}" />
-  <xacro:property name="r_elbow_flex_joint_upper"        value="${r*c['joints']['r_elbow_flex_joint']['minGoal']}" />
+  <xacro:property name="r_elbow_flex_joint_lower"        value="0" />
+  <xacro:property name="r_elbow_flex_joint_upper"        value="${r*(c['joints']['r_elbow_flex_joint']['minGoal'] - c['joints']['r_elbow_flex_joint']['maxGoal'])}" />
   <xacro:property name="r_elbow_flex_joint_velocity"     value="${r*c['joints']['r_elbow_flex_joint']['maxSpeed']}" />
   <xacro:property name="eyes_pan_joint_lower"            value="${r*c['joints']['eyes_pan_joint']['minGoal']}" />
@@ -68,6 +68,6 @@
   <xacro:property name="r_pinky_joint_upper"             value="${r*c['joints']['r_pinky_joint']['maxGoal']}" />
   <xacro:property name="r_pinky_joint_velocity"          value="${r*c['joints']['r_pinky_joint']['maxSpeed']}" />
-  <xacro:property name="l_shoulder_out_joint_lower"      value="${r*c['joints']['l_shoulder_out_joint']['minGoal']}" />
-  <xacro:property name="l_shoulder_out_joint_upper"      value="${r*c['joints']['l_shoulder_out_joint']['maxGoal']}" />
+  <xacro:property name="l_shoulder_out_joint_lower"      value="0" />
+  <xacro:property name="l_shoulder_out_joint_upper"      value="${r*(c['joints']['l_shoulder_out_joint']['maxGoal'] - c['joints']['l_shoulder_out_joint']['minGoal'])}" />
   <xacro:property name="l_shoulder_out_joint_velocity"   value="${r*c['joints']['l_shoulder_out_joint']['maxSpeed']}" />
   <xacro:property name="waist_pan_joint_lower"           value="${r*c['joints']['waist_pan_joint']['minGoal']}" />
@@ -86,6 +86,6 @@
   <xacro:property name="head_tilt_joint_upper"           value="${r*c['joints']['head_tilt_joint']['maxGoal']}" />
   <xacro:property name="head_tilt_joint_velocity"        value="${r*c['joints']['head_tilt_joint']['maxSpeed']}" />
-  <xacro:property name="r_shoulder_out_joint_lower"      value="${-r*c['joints']['r_shoulder_out_joint']['minGoal']}" />
-  <xacro:property name="r_shoulder_out_joint_upper"      value="${-r*c['joints']['r_shoulder_out_joint']['maxGoal']}" />
+  <xacro:property name="r_shoulder_out_joint_lower"      value="0" />
+  <xacro:property name="r_shoulder_out_joint_upper"      value="${r*(c['joints']['r_shoulder_out_joint']['minGoal'] - c['joints']['r_shoulder_out_joint']['maxGoal'])}" />
   <xacro:property name="r_shoulder_out_joint_velocity"   value="${r*c['joints']['r_shoulder_out_joint']['maxSpeed']}" />
 </robot>
