Commit message: elbow_flex: negate the axis too, so the MODEL bends the right way
My bug, from the re-base in the previous commit. Moving the elbow range from
[-1.396, -0.262] to [0, 1.134] flipped the sign of the joint value, so flexing changed from
1.134 rad NEGATIVE about +Y to 1.134 rad POSITIVE about +Y -- the opposite rotation.

The driver was corrected for that (invert flipped) so the real robot moved correctly, which
is exactly what made it easy to miss: Simon saw the robot doing the right thing while RViz
bent the elbows BACKWARDS, into a pose a human arm cannot reach.

Negating the axis restores the original rotation for the new positive values. The joint
value convention is unchanged, so the driver mapping and the servo behaviour stay exactly
as they are -- only the model's direction of rotation changes.

Checked the other joints touched today for the same class of mistake and they are clean:
shoulder_out was a SHIFT of an already-positive range (direction preserved), and
shoulder_lift and wrist_roll had their axis AND limits negated together, which cancels.
The elbow was the only one where the limits moved without the axis following.

Co-Authored-By: Claude Opus 5 (1M context) <noreply@anthropic.com>
Claude-Session: https://claude.ai/code/session_01Kpk5vJ7u2Qct1dnDk8Kg4X

File: inmoov_description/urdf/asmArm.urdf.xacro (robot description, xacro)
@@ -122,5 +122,5 @@
   </joint>
   <joint name="${side}_elbow_flex_joint" type="revolute">
-    <axis xyz="0 1 0"/>
+    <axis xyz="0 -1 0"/>
     <xacro:if value="${side == 'l'}">
       <limit effort="10000.0" lower="${l_elbow_flex_joint_lower}" upper="${l_elbow_flex_joint_upper}" velocity="${l_elbow_flex_joint_velocity}" />

Commit message: l_upper_arm_roll: side-dependent axis so RViz agrees with the robot
Simon: "the robot moves correctly but the URDF goes the opposite". Same class of mistake as
the elbow -- the driver was corrected earlier by flipping this joint's invert flag, and the
model was never touched, so RViz has been rotating the left bicep the wrong way since.

The axis was a single line in the shared ${side} macro, applied identically to both arms. It
is now side-dependent (left 0 0 -1, right 0 0 1), the same way the limits already were.

That also closes the last real mirroring gap. The symmetry check wanted a_R == -M a_L; both
sides were (0,0,1) with the right required to be (0,0,-1). Negating the LEFT satisfies it
equally: -M(0,0,-1) == (0,0,1). So the pair now moves in mirror image for the same slider
position, which is what Simon asked for two commits ago.

The joint value convention is untouched (symmetric limits, home 0), so the driver mapping
and the servo behaviour are unchanged -- the robot keeps doing what it already did right.

Remaining unmirrored per the checker: pinky1, ring1, thumb1. Those are geometry-only finger
sub-links with one tendon servo behind each finger, and Simon has confirmed the fingers work
correctly on the robot. Left alone deliberately.

Co-Authored-By: Claude Opus 5 (1M context) <noreply@anthropic.com>
Claude-Session: https://claude.ai/code/session_01Kpk5vJ7u2Qct1dnDk8Kg4X

File: inmoov_description/urdf/asmArm.urdf.xacro (robot description, xacro)
@@ -110,5 +110,13 @@
   </joint>
   <joint name="${side}_upper_arm_roll_joint" type="revolute">
-    <axis xyz="0 0 1"/>
+    <!-- Side-dependent axis. The left bicep rotates the opposite way to the right for the
+         same joint value, so mirroring it here keeps RViz agreeing with the real robot AND
+         makes the pair move in mirror image for the same slider position. -->
+    <xacro:if value="${side == 'l'}">
+      <axis xyz="0 0 -1"/>
+    </xacro:if>
+    <xacro:if value="${side == 'r'}">
+      <axis xyz="0 0 1"/>
+    </xacro:if>
     <xacro:if value="${side == 'l'}">
       <limit effort="10000.0" lower="${l_upper_arm_roll_joint_lower}" upper="${l_upper_arm_roll_joint_upper}" velocity="${l_upper_arm_roll_joint_velocity}" />
