Commit message: Working, lots of work to clean up

File: inmoov_description/urdf/config.inertial.urdf.xacro (robot description, xacro)
@@ -12,5 +12,5 @@
   <xacro:property name="id" value="${ md * md * md}"/>
 <!--
-Opened mesh /home/grey/inmoov_ros/src/inmoov_ros/inmoov_meshes/meshes/bicep.stl in 6 msec
+Opened mesh /home/grey/inmoov_ros/src/inmoov_ros/inmoov_description/meshes/bicep.stl in 6 msec
 All files opened in 2436 msec
 Mesh Bounding Box Size 108.018005 91.844795 231.879486
@@ -45,5 +45,5 @@
   </xacro:macro>
 <!--
-Opened mesh /home/grey/inmoov_ros/src/inmoov_ros/inmoov_meshes/meshes/bicepcover.stl in 18 msec
+Opened mesh /home/grey/inmoov_ros/src/inmoov_ros/inmoov_description/meshes/bicepcover.stl in 18 msec
 All files opened in 2233 msec
 Mesh Bounding Box Size 129.930206 91.769051 208.188858
@@ -78,5 +78,5 @@
   </xacro:macro>
 <!--
-Opened mesh /home/grey/inmoov_ros/src/inmoov_ros/inmoov_meshes/meshes/camera.stl in 8 msec
+Opened mesh /home/grey/inmoov_ros/src/inmoov_ros/inmoov_description/meshes/camera.stl in 8 msec
 All files opened in 2697 msec
 Mesh Bounding Box Size 8.000001 33.499996 19.499996
@@ -111,5 +111,5 @@
   </xacro:macro>
 <!--
-Opened mesh /home/grey/inmoov_ros/src/inmoov_ros/inmoov_meshes/meshes/chest.stl in 50 msec
+Opened mesh /home/grey/inmoov_ros/src/inmoov_ros/inmoov_description/meshes/chest.stl in 50 msec
 All files opened in 1996 msec
 Mesh Bounding Box Size 80.510498 307.491943 275.934937
@@ -144,5 +144,5 @@
   </xacro:macro>
 <!--
-Opened mesh /home/grey/inmoov_ros/src/inmoov_ros/inmoov_meshes/meshes/disk.stl in 17 msec
+Opened mesh /home/grey/inmoov_ros/src/inmoov_ros/inmoov_description/meshes/disk.stl in 17 msec
 All files opened in 2305 msec
 Mesh Bounding Box Size 32.199123 141.520432 141.527847
@@ -177,5 +177,5 @@
   </xacro:macro>
 <!--
-Opened mesh /home/grey/inmoov_ros/src/inmoov_ros/inmoov_meshes/meshes/earleftv1.stl in 22 msec
+Opened mesh /home/grey/inmoov_ros/src/inmoov_ros/inmoov_description/meshes/earleftv1.stl in 22 msec
 All files opened in 2362 msec
 Mesh Bounding Box Size 91.007996 25.182009 91.007942
@@ -210,5 +210,5 @@
   </xacro:macro>
 <!--
-Opened mesh /home/grey/inmoov_ros/src/inmoov_ros/inmoov_meshes/meshes/earrightv1.stl in 185 msec
+Opened mesh /home/grey/inmoov_ros/src/inmoov_ros/inmoov_description/meshes/earrightv1.stl in 185 msec
 All files opened in 2114 msec
 Mesh Bounding Box Size 91.014008 25.182001 91.013977
@@ -243,5 +243,5 @@
   </xacro:macro>
 <!--
-Opened mesh /home/grey/inmoov_ros/src/inmoov_ros/inmoov_meshes/meshes/eye.stl in 3 msec
+Opened mesh /home/grey/inmoov_ros/src/inmoov_ros/inmoov_description/meshes/eye.stl in 3 msec
 All files opened in 1580 msec
 Mesh Bounding Box Size 8.000001 36.000000 35.969540
@@ -276,5 +276,5 @@
   </xacro:macro>
 <!--
-Opened mesh /home/grey/inmoov_ros/src/inmoov_ros/inmoov_meshes/meshes/eyesupport.stl in 2 msec
+Opened mesh /home/grey/inmoov_ros/src/inmoov_ros/inmoov_description/meshes/eyesupport.stl in 2 msec
 All files opened in 1536 msec
 Mesh Bounding Box Size 33.271500 76.999481 75.081680
@@ -309,5 +309,5 @@
   </xacro:macro>
 <!--
-Opened mesh /home/grey/inmoov_ros/src/inmoov_ros/inmoov_meshes/meshes/face.stl in 4 msec
+Opened mesh /home/grey/inmoov_ros/src/inmoov_ros/inmoov_description/meshes/face.stl in 4 msec
 All files opened in 1547 msec
 Mesh Bounding Box Size 58.885715 130.552460 65.225174
@@ -342,5 +342,5 @@
   </xacro:macro>
 <!--
-Opened mesh /home/grey/inmoov_ros/src/inmoov_ros/inmoov_meshes/meshes/head.stl in 3 msec
+Opened mesh /home/grey/inmoov_ros/src/inmoov_ros/inmoov_description/meshes/head.stl in 3 msec
 All files opened in 1403 msec
 Mesh Bounding Box Size 148.349350 130.531616 66.729294
@@ -375,5 +375,5 @@
   </xacro:macro>
 <!--
-Opened mesh /home/grey/inmoov_ros/src/inmoov_ros/inmoov_meshes/meshes/head_base.stl in 6 msec
+Opened mesh /home/grey/inmoov_ros/src/inmoov_ros/inmoov_description/meshes/head_base.stl in 6 msec
 All files opened in 1357 msec
 Mesh Bounding Box Size 69.337830 92.601379 32.000000
@@ -408,5 +408,5 @@
   </xacro:macro>
 <!--
-Opened mesh /home/grey/inmoov_ros/src/inmoov_ros/inmoov_meshes/meshes/index3_1.stl in 2 msec
+Opened mesh /home/grey/inmoov_ros/src/inmoov_ros/inmoov_description/meshes/index3_1.stl in 2 msec
 All files opened in 1522 msec
 Mesh Bounding Box Size 17.238571 17.350281 48.785606
@@ -441,5 +441,5 @@
   </xacro:macro>
 <!--
-Opened mesh /home/grey/inmoov_ros/src/inmoov_ros/inmoov_meshes/meshes/index3_2.stl in 7 msec
+Opened mesh /home/grey/inmoov_ros/src/inmoov_ros/inmoov_description/meshes/index3_2.stl in 7 msec
 All files opened in 1581 msec
 Mesh Bounding Box Size 16.419373 15.360427 34.058228
@@ -474,5 +474,5 @@
   </xacro:macro>
 <!--
-Opened mesh /home/grey/inmoov_ros/src/inmoov_ros/inmoov_meshes/meshes/index3_3.stl in 3 msec
+Opened mesh /home/grey/inmoov_ros/src/inmoov_ros/inmoov_description/meshes/index3_3.stl in 3 msec
 All files opened in 1481 msec
 Mesh Bounding Box Size 15.530320 14.615662 35.068295
@@ -507,5 +507,5 @@
   </xacro:macro>
 <!--
-Opened mesh /home/grey/inmoov_ros/src/inmoov_ros/inmoov_meshes/meshes/iris.stl in 7 msec
+Opened mesh /home/grey/inmoov_ros/src/inmoov_ros/inmoov_description/meshes/iris.stl in 7 msec
 All files opened in 1708 msec
 Mesh Bounding Box Size 4.850000 21.782320 21.764652
@@ -540,5 +540,5 @@
   </xacro:macro>
 <!--
-Opened mesh /home/grey/inmoov_ros/src/inmoov_ros/inmoov_meshes/meshes/jaw.stl in 3 msec
+Opened mesh /home/grey/inmoov_ros/src/inmoov_ros/inmoov_description/meshes/jaw.stl in 3 msec
 All files opened in 1932 msec
 Mesh Bounding Box Size 151.468292 113.023956 114.478699
@@ -573,5 +573,5 @@
   </xacro:macro>
 <!--
-Opened mesh /home/grey/inmoov_ros/src/inmoov_ros/inmoov_meshes/meshes/kinectone.stl in 6 msec
+Opened mesh /home/grey/inmoov_ros/src/inmoov_ros/inmoov_description/meshes/kinectone.stl in 6 msec
 All files opened in 1236 msec
 Mesh Bounding Box Size 250.000031 82.000008 64.499985
@@ -606,5 +606,5 @@
   </xacro:macro>
 <!--
-Opened mesh /home/grey/inmoov_ros/src/inmoov_ros/inmoov_meshes/meshes/l_cover_hand.stl in 32 msec
+Opened mesh /home/grey/inmoov_ros/src/inmoov_ros/inmoov_description/meshes/l_cover_hand.stl in 32 msec
 All files opened in 1460 msec
 Mesh Bounding Box Size 13.736001 84.862000 108.330002
@@ -639,5 +639,5 @@
   </xacro:macro>
 <!--
-Opened mesh /home/grey/inmoov_ros/src/inmoov_ros/inmoov_meshes/meshes/l_cover_handpinky.stl in 6 msec
+Opened mesh /home/grey/inmoov_ros/src/inmoov_ros/inmoov_description/meshes/l_cover_handpinky.stl in 6 msec
 All files opened in 1500 msec
 Mesh Bounding Box Size 5.456001 32.141998 56.658005
@@ -672,5 +672,5 @@
   </xacro:macro>
 <!--
-Opened mesh /home/grey/inmoov_ros/src/inmoov_ros/inmoov_meshes/meshes/l_cover_handring.stl in 17 msec
+Opened mesh /home/grey/inmoov_ros/src/inmoov_ros/inmoov_description/meshes/l_cover_handring.stl in 17 msec
 All files opened in 2914 msec
 Mesh Bounding Box Size 6.642000 33.834000 43.076000
@@ -705,5 +705,5 @@
   </xacro:macro>
 <!--
-Opened mesh /home/grey/inmoov_ros/src/inmoov_ros/inmoov_meshes/meshes/l_cover_index.stl in 8 msec
+Opened mesh /home/grey/inmoov_ros/src/inmoov_ros/inmoov_description/meshes/l_cover_index.stl in 8 msec
 All files opened in 1384 msec
 Mesh Bounding Box Size 8.594393 17.415220 35.119446
@@ -738,5 +738,5 @@
   </xacro:macro>
 <!--
-Opened mesh /home/grey/inmoov_ros/src/inmoov_ros/inmoov_meshes/meshes/l_cover_middle.stl in 6 msec
+Opened mesh /home/grey/inmoov_ros/src/inmoov_ros/inmoov_description/meshes/l_cover_middle.stl in 6 msec
 All files opened in 1439 msec
 Mesh Bounding Box Size 8.813518 18.337889 38.744076
@@ -771,5 +771,5 @@
   </xacro:macro>
 <!--
-Opened mesh /home/grey/inmoov_ros/src/inmoov_ros/inmoov_meshes/meshes/l_cover_pinky.stl in 7 msec
+Opened mesh /home/grey/inmoov_ros/src/inmoov_ros/inmoov_description/meshes/l_cover_pinky.stl in 7 msec
 All files opened in 1484 msec
 Mesh Bounding Box Size 7.799893 16.734661 33.440189
@@ -804,5 +804,5 @@
   </xacro:macro>
 <!--
-Opened mesh /home/grey/inmoov_ros/src/inmoov_ros/inmoov_meshes/meshes/l_cover_ring.stl in 5 msec
+Opened mesh /home/grey/inmoov_ros/src/inmoov_ros/inmoov_description/meshes/l_cover_ring.stl in 5 msec
 All files opened in 1463 msec
 Mesh Bounding Box Size 8.088491 17.430080 36.716965
@@ -837,5 +837,5 @@
   </xacro:macro>
 <!--
-Opened mesh /home/grey/inmoov_ros/src/inmoov_ros/inmoov_meshes/meshes/l_cover_thumb.stl in 4 msec
+Opened mesh /home/grey/inmoov_ros/src/inmoov_ros/inmoov_description/meshes/l_cover_thumb.stl in 4 msec
 All files opened in 1596 msec
 Mesh Bounding Box Size 6.319447 26.349285 49.800488
@@ -870,5 +870,5 @@
   </xacro:macro>
 <!--
-Opened mesh /home/grey/inmoov_ros/src/inmoov_ros/inmoov_meshes/meshes/l_eyesupport.stl in 2 msec
+Opened mesh /home/grey/inmoov_ros/src/inmoov_ros/inmoov_description/meshes/l_eyesupport.stl in 2 msec
 All files opened in 1191 msec
 Mesh Bounding Box Size 14.000004 35.808380 45.097652
@@ -903,5 +903,5 @@
   </xacro:macro>
 <!--
-Opened mesh /home/grey/inmoov_ros/src/inmoov_ros/inmoov_meshes/meshes/l_forearm.stl in 16 msec
+Opened mesh /home/grey/inmoov_ros/src/inmoov_ros/inmoov_description/meshes/l_forearm.stl in 16 msec
 All files opened in 1710 msec
 Mesh Bounding Box Size 108.761078 103.942200 315.046661
@@ -936,5 +936,5 @@
   </xacro:macro>
 <!--
-Opened mesh /home/grey/inmoov_ros/src/inmoov_ros/inmoov_meshes/meshes/l_hand.stl in 12 msec
+Opened mesh /home/grey/inmoov_ros/src/inmoov_ros/inmoov_description/meshes/l_hand.stl in 12 msec
 All files opened in 2042 msec
 Mesh Bounding Box Size 44.331417 93.143219 128.509338
@@ -969,5 +969,5 @@
   </xacro:macro>
 <!--
-Opened mesh /home/grey/inmoov_ros/src/inmoov_ros/inmoov_meshes/meshes/l_pinky3_1.stl in 12 msec
+Opened mesh /home/grey/inmoov_ros/src/inmoov_ros/inmoov_description/meshes/l_pinky3_1.stl in 12 msec
 All files opened in 1582 msec
 Mesh Bounding Box Size 17.696007 58.876789 43.411186
@@ -1002,5 +1002,5 @@
   </xacro:macro>
 <!--
-Opened mesh /home/grey/inmoov_ros/src/inmoov_ros/inmoov_meshes/meshes/l_ring3_1.stl in 2 msec
+Opened mesh /home/grey/inmoov_ros/src/inmoov_ros/inmoov_description/meshes/l_ring3_1.stl in 2 msec
 All files opened in 1673 msec
 Mesh Bounding Box Size 17.686001 48.905632 38.091835
@@ -1035,5 +1035,5 @@
   </xacro:macro>
 <!--
-Opened mesh /home/grey/inmoov_ros/src/inmoov_ros/inmoov_meshes/meshes/l_shoulder.stl in 5 msec
+Opened mesh /home/grey/inmoov_ros/src/inmoov_ros/inmoov_description/meshes/l_shoulder.stl in 5 msec
 All files opened in 1242 msec
 Mesh Bounding Box Size 102.575752 111.850540 126.307632
@@ -1068,5 +1068,5 @@
   </xacro:macro>
 <!--
-Opened mesh /home/grey/inmoov_ros/src/inmoov_ros/inmoov_meshes/meshes/l_shoulder_base.stl in 7 msec
+Opened mesh /home/grey/inmoov_ros/src/inmoov_ros/inmoov_description/meshes/l_shoulder_base.stl in 7 msec
 All files opened in 2182 msec
 Mesh Bounding Box Size 102.761749 110.730751 118.874138
@@ -1101,5 +1101,5 @@
   </xacro:macro>
 <!--
-Opened mesh /home/grey/inmoov_ros/src/inmoov_ros/inmoov_meshes/meshes/l_thumb5_1.stl in 5 msec
+Opened mesh /home/grey/inmoov_ros/src/inmoov_ros/inmoov_description/meshes/l_thumb5_1.stl in 5 msec
 All files opened in 1492 msec
 Mesh Bounding Box Size 22.555820 43.031254 35.923035
@@ -1134,5 +1134,5 @@
   </xacro:macro>
 <!--
-Opened mesh /home/grey/inmoov_ros/src/inmoov_ros/inmoov_meshes/meshes/middle3_1.stl in 2 msec
+Opened mesh /home/grey/inmoov_ros/src/inmoov_ros/inmoov_description/meshes/middle3_1.stl in 2 msec
 All files opened in 1320 msec
 Mesh Bounding Box Size 18.482727 18.602509 52.306591
@@ -1167,5 +1167,5 @@
   </xacro:macro>
 <!--
-Opened mesh /home/grey/inmoov_ros/src/inmoov_ros/inmoov_meshes/meshes/middle3_2.stl in 4 msec
+Opened mesh /home/grey/inmoov_ros/src/inmoov_ros/inmoov_description/meshes/middle3_2.stl in 4 msec
 All files opened in 1454 msec
 Mesh Bounding Box Size 17.604366 16.469009 36.516296
@@ -1200,5 +1200,5 @@
   </xacro:macro>
 <!--
-Opened mesh /home/grey/inmoov_ros/src/inmoov_ros/inmoov_meshes/meshes/middle3_3.stl in 3 msec
+Opened mesh /home/grey/inmoov_ros/src/inmoov_ros/inmoov_description/meshes/middle3_3.stl in 3 msec
 All files opened in 1329 msec
 Mesh Bounding Box Size 16.651167 15.670519 37.599258
@@ -1233,5 +1233,5 @@
   </xacro:macro>
 <!--
-Opened mesh /home/grey/inmoov_ros/src/inmoov_ros/inmoov_meshes/meshes/mid_stomach.stl in 12 msec
+Opened mesh /home/grey/inmoov_ros/src/inmoov_ros/inmoov_description/meshes/mid_stomach.stl in 12 msec
 All files opened in 1561 msec
 Mesh Bounding Box Size 171.763184 295.432159 172.122498
@@ -1266,5 +1266,5 @@
   </xacro:macro>
 <!--
-Opened mesh /home/grey/inmoov_ros/src/inmoov_ros/inmoov_meshes/meshes/pinky3_2.stl in 4 msec
+Opened mesh /home/grey/inmoov_ros/src/inmoov_ros/inmoov_description/meshes/pinky3_2.stl in 4 msec
 All files opened in 2164 msec
 Mesh Bounding Box Size 14.813997 14.910004 41.924004
@@ -1299,5 +1299,5 @@
   </xacro:macro>
 <!--
-Opened mesh /home/grey/inmoov_ros/src/inmoov_ros/inmoov_meshes/meshes/pinky3_3.stl in 4 msec
+Opened mesh /home/grey/inmoov_ros/src/inmoov_ros/inmoov_description/meshes/pinky3_3.stl in 4 msec
 All files opened in 2273 msec
 Mesh Bounding Box Size 14.109985 13.200013 29.268002
@@ -1332,5 +1332,5 @@
   </xacro:macro>
 <!--
-Opened mesh /home/grey/inmoov_ros/src/inmoov_ros/inmoov_meshes/meshes/pinky3_4.stl in 9 msec
+Opened mesh /home/grey/inmoov_ros/src/inmoov_ros/inmoov_description/meshes/pinky3_4.stl in 9 msec
 All files opened in 1721 msec
 Mesh Bounding Box Size 13.346009 12.559998 30.136002
@@ -1365,5 +1365,5 @@
   </xacro:macro>
 <!--
-Opened mesh /home/grey/inmoov_ros/src/inmoov_ros/inmoov_meshes/meshes/r_cover_hand.stl in 31 msec
+Opened mesh /home/grey/inmoov_ros/src/inmoov_ros/inmoov_description/meshes/r_cover_hand.stl in 31 msec
 All files opened in 1286 msec
 Mesh Bounding Box Size 13.736000 84.862000 108.330017
@@ -1398,5 +1398,5 @@
   </xacro:macro>
 <!--
-Opened mesh /home/grey/inmoov_ros/src/inmoov_ros/inmoov_meshes/meshes/r_cover_handpinky.stl in 8 msec
+Opened mesh /home/grey/inmoov_ros/src/inmoov_ros/inmoov_description/meshes/r_cover_handpinky.stl in 8 msec
 All files opened in 1616 msec
 Mesh Bounding Box Size 5.456001 32.141998 56.658005
@@ -1431,5 +1431,5 @@
   </xacro:macro>
 <!--
-Opened mesh /home/grey/inmoov_ros/src/inmoov_ros/inmoov_meshes/meshes/r_cover_handring.stl in 9 msec
+Opened mesh /home/grey/inmoov_ros/src/inmoov_ros/inmoov_description/meshes/r_cover_handring.stl in 9 msec
 All files opened in 1687 msec
 Mesh Bounding Box Size 6.641999 33.834000 43.076000
@@ -1464,5 +1464,5 @@
   </xacro:macro>
 <!--
-Opened mesh /home/grey/inmoov_ros/src/inmoov_ros/inmoov_meshes/meshes/r_cover_index.stl in 7 msec
+Opened mesh /home/grey/inmoov_ros/src/inmoov_ros/inmoov_description/meshes/r_cover_index.stl in 7 msec
 All files opened in 1714 msec
 Mesh Bounding Box Size 8.594393 17.415220 35.119446
@@ -1497,5 +1497,5 @@
   </xacro:macro>
 <!--
-Opened mesh /home/grey/inmoov_ros/src/inmoov_ros/inmoov_meshes/meshes/r_cover_middle.stl in 22 msec
+Opened mesh /home/grey/inmoov_ros/src/inmoov_ros/inmoov_description/meshes/r_cover_middle.stl in 22 msec
 All files opened in 1370 msec
 Mesh Bounding Box Size 8.813518 18.337889 38.744076
@@ -1530,5 +1530,5 @@
   </xacro:macro>
 <!--
-Opened mesh /home/grey/inmoov_ros/src/inmoov_ros/inmoov_meshes/meshes/r_cover_pinky.stl in 25 msec
+Opened mesh /home/grey/inmoov_ros/src/inmoov_ros/inmoov_description/meshes/r_cover_pinky.stl in 25 msec
 All files opened in 1370 msec
 Mesh Bounding Box Size 7.799893 16.734661 33.440189
@@ -1563,5 +1563,5 @@
   </xacro:macro>
 <!--
-Opened mesh /home/grey/inmoov_ros/src/inmoov_ros/inmoov_meshes/meshes/r_cover_ring.stl in 24 msec
+Opened mesh /home/grey/inmoov_ros/src/inmoov_ros/inmoov_description/meshes/r_cover_ring.stl in 24 msec
 All files opened in 1487 msec
 Mesh Bounding Box Size 8.088491 17.430080 36.716965
@@ -1596,5 +1596,5 @@
   </xacro:macro>
 <!--
-Opened mesh /home/grey/inmoov_ros/src/inmoov_ros/inmoov_meshes/meshes/r_cover_thumb.stl in 21 msec
+Opened mesh /home/grey/inmoov_ros/src/inmoov_ros/inmoov_description/meshes/r_cover_thumb.stl in 21 msec
 All files opened in 1387 msec
 Mesh Bounding Box Size 6.319447 26.349291 49.800488
@@ -1629,5 +1629,5 @@
   </xacro:macro>
 <!--
-Opened mesh /home/grey/inmoov_ros/src/inmoov_ros/inmoov_meshes/meshes/r_eyesupport.stl in 2 msec
+Opened mesh /home/grey/inmoov_ros/src/inmoov_ros/inmoov_description/meshes/r_eyesupport.stl in 2 msec
 All files opened in 1164 msec
 Mesh Bounding Box Size 14.000004 35.808380 45.097652
@@ -1662,5 +1662,5 @@
   </xacro:macro>
 <!--
-Opened mesh /home/grey/inmoov_ros/src/inmoov_ros/inmoov_meshes/meshes/r_forearm.stl in 9 msec
+Opened mesh /home/grey/inmoov_ros/src/inmoov_ros/inmoov_description/meshes/r_forearm.stl in 9 msec
 All files opened in 1247 msec
 Mesh Bounding Box Size 108.761078 103.942200 315.046661
@@ -1695,5 +1695,5 @@
   </xacro:macro>
 <!--
-Opened mesh /home/grey/inmoov_ros/src/inmoov_ros/inmoov_meshes/meshes/r_hand.stl in 14 msec
+Opened mesh /home/grey/inmoov_ros/src/inmoov_ros/inmoov_description/meshes/r_hand.stl in 14 msec
 All files opened in 1521 msec
 Mesh Bounding Box Size 44.331417 93.143219 128.509323
@@ -1728,5 +1728,5 @@
   </xacro:macro>
 <!--
-Opened mesh /home/grey/inmoov_ros/src/inmoov_ros/inmoov_meshes/meshes/ring3_2.stl in 5 msec
+Opened mesh /home/grey/inmoov_ros/src/inmoov_ros/inmoov_description/meshes/ring3_2.stl in 5 msec
 All files opened in 1503 msec
 Mesh Bounding Box Size 16.450043 16.556625 46.554031
@@ -1761,5 +1761,5 @@
   </xacro:macro>
 <!--
-Opened mesh /home/grey/inmoov_ros/src/inmoov_ros/inmoov_meshes/meshes/ring3_3.stl in 2 msec
+Opened mesh /home/grey/inmoov_ros/src/inmoov_ros/inmoov_description/meshes/ring3_3.stl in 2 msec
 All files opened in 1562 msec
 Mesh Bounding Box Size 15.668304 14.657790 32.500313
@@ -1794,5 +1794,5 @@
   </xacro:macro>
 <!--
-Opened mesh /home/grey/inmoov_ros/src/inmoov_ros/inmoov_meshes/meshes/ring3_4.stl in 2 msec
+Opened mesh /home/grey/inmoov_ros/src/inmoov_ros/inmoov_description/meshes/ring3_4.stl in 2 msec
 All files opened in 1837 msec
 Mesh Bounding Box Size 14.819916 13.947111 33.464180
@@ -1827,5 +1827,5 @@
   </xacro:macro>
 <!--
-Opened mesh /home/grey/inmoov_ros/src/inmoov_ros/inmoov_meshes/meshes/r_pinky3_1.stl in 9 msec
+Opened mesh /home/grey/inmoov_ros/src/inmoov_ros/inmoov_description/meshes/r_pinky3_1.stl in 9 msec
 All files opened in 2265 msec
 Mesh Bounding Box Size 17.696005 58.876789 43.411186
@@ -1860,5 +1860,5 @@
   </xacro:macro>
 <!--
-Opened mesh /home/grey/inmoov_ros/src/inmoov_ros/inmoov_meshes/meshes/r_ring3_1.stl in 6 msec
+Opened mesh /home/grey/inmoov_ros/src/inmoov_ros/inmoov_description/meshes/r_ring3_1.stl in 6 msec
 All files opened in 1388 msec
 Mesh Bounding Box Size 17.686001 48.905632 38.091835
@@ -1893,5 +1893,5 @@
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