Commit message: Gazebo / RVIZ render but nothing moves

File: inmoov_description/robots/inmoov.urdf.xacro (robot description, xacro)
@@ -4,14 +4,14 @@
 <xacro:include filename="$(find inmoov_description)/urdf/config.inertial.urdf.xacro" />
 <xacro:include filename="$(find inmoov_description)/urdf/materials.urdf.xacro" />
+<xacro:include filename="$(find inmoov_description)/urdf/asmBase.urdf.xacro" />
+<xacro:include filename="$(find inmoov_description)/urdf/asmTorso.urdf.xacro" />
+<xacro:include filename="$(find inmoov_description)/urdf/asmHead.urdf.xacro" />
+<xacro:include filename="$(find inmoov_description)/urdf/asmEye.urdf.xacro" />
+<xacro:include filename="$(find inmoov_description)/urdf/asmFace.urdf.xacro" />
+<xacro:include filename="$(find inmoov_description)/urdf/asmArm.urdf.xacro" />
+<xacro:include filename="$(find inmoov_description)/urdf/asmHand.urdf.xacro" />
 <xacro:include filename="$(find inmoov_description)/urdf/inmoov.gazebo" />
-  <xacro:include filename="$(find inmoov_description)/urdf/materials.urdf.xacro" />
-  <xacro:include filename="$(find inmoov_description)/urdf/asmBase.urdf.xacro" />
-  <xacro:include filename="$(find inmoov_description)/urdf/asmTorso.urdf.xacro" />
-  <xacro:include filename="$(find inmoov_description)/urdf/asmHead.urdf.xacro" />
-  <xacro:include filename="$(find inmoov_description)/urdf/asmEye.urdf.xacro" />
-  <xacro:include filename="$(find inmoov_description)/urdf/asmFace.urdf.xacro" />
-  <xacro:include filename="$(find inmoov_description)/urdf/asmArm.urdf.xacro" />
-  <xacro:include filename="$(find inmoov_description)/urdf/asmHand.urdf.xacro" />
   <link name="world"/>
+    <xacro:virtual_inertial/>
   <joint name="fixed" type="fixed">
     <parent link="world"/>
@@ -26,5 +26,11 @@
       <xacro:base_color/>
     </visual>
-  </link>
+    <collision>
+      <geometry>
+        <cylinder length="0.11" radius="0.26"/>
+      </geometry>
+      <origin rpy="0 0 0" xyz="0 0 0.055"/>
+    </collision>
+</link>
   <joint name="base_to_pedestal_link" type="fixed">
     <parent link="base_link"/>
@@ -33,4 +39,5 @@
   </joint>
   <link name="pedestal_link">
+    <xacro:virtual_inertial/>
     <visual>
       <geometry>
@@ -40,5 +47,11 @@
       <xacro:base_color/>
     </visual>
-  </link>
+    <collision>
+      <geometry>
+        <cylinder length="0.94" radius="0.0254"/>
+      </geometry>
+      <origin rpy="0 0 0" xyz="0 0 0.58"/>
+    </collision>
+</link>
   <link name="head_tilt_link">
     <visual>
@@ -50,5 +63,11 @@
     </visual>
     <xacro:virtual_inertial/>
-  </link>
+    <collision>
+      <geometry>
+        <mesh filename="package://inmoov_description/meshes/virtual.stl" scale="0.001 0.001 0.001"/>
+      </geometry>
+      <origin rpy="0 0 3.1415" xyz="0 0 0"/>
+    </collision>
+</link>
   <joint name="pedestal_to_mid_stomach_joint" type="fixed">
     <parent link="pedestal_link"/>

File: inmoov_description/urdf/asmArm.urdf.xacro (robot description, xacro)
@@ -16,5 +16,11 @@
       <xacro:r_shoulder_base_inertial/>
     </xacro:if>
-  </link>
+    <collision>
+      <geometry>
+        <mesh filename="package://inmoov_description/meshes/${side}_shoulder_base.stl" scale="0.001 0.001 0.001"/>
+      </geometry>
+      <origin rpy="0 0 0" xyz="0 0 0"/>
+    </collision>
+</link>
   <link name="${side}_shoulder_link">
     <visual>
@@ -31,5 +37,11 @@
       <xacro:r_shoulder_inertial/>
     </xacro:if>
-  </link>
+    <collision>
+      <geometry>
+        <mesh filename="package://inmoov_description/meshes/${side}_shoulder.stl" scale="0.001 0.001 0.001"/>
+      </geometry>
+      <origin rpy="0 0 0" xyz="0 0 0"/>
+    </collision>
+</link>
   <link name="${side}_bicep_link">
     <visual>
@@ -41,5 +53,11 @@
     </visual>
     <xacro:bicep_inertial/>
-  </link>
+    <collision>
+      <geometry>
+        <mesh filename="package://inmoov_description/meshes/bicep.stl" scale="0.001 0.001 0.001"/>
+      </geometry>
+      <origin rpy="0 0 0" xyz="0 0 0"/>
+    </collision>
+</link>
   <link name="${side}_bicepcover_link">
     <visual>
@@ -51,5 +69,11 @@
     </visual>
     <xacro:bicepcover_inertial/>
-  </link>
+    <collision>
+      <geometry>
+        <mesh filename="package://inmoov_description/meshes/bicepcover.stl" scale="0.001 0.001 0.001"/>
+      </geometry>
+      <origin rpy="0 0 0" xyz="0 0 0"/>
+    </collision>
+</link>
   <link name="${side}_forearm_link">
     <visual>
@@ -66,5 +90,11 @@
       <xacro:r_forearm_inertial/>
     </xacro:if>
-  </link>
+    <collision>
+      <geometry>
+        <mesh filename="package://inmoov_description/meshes/${side}_forearm.stl" scale="0.001 0.001 0.001"/>
+      </geometry>
+      <origin rpy="0 0 0" xyz="${flip * 0.001} 0 0"/>
+    </collision>
+</link>
   <joint name="${side}_shoulder_lift_joint" type="revolute">
     <axis xyz="0 1 0"/>

File: inmoov_description/urdf/asmEye.urdf.xacro (robot description, xacro)
@@ -16,5 +16,11 @@
       <xacro:r_eyesupport_inertial/>
     </xacro:if>
-  </link>
+    <collision>
+      <geometry>
+        <mesh filename="package://inmoov_description/meshes/${side}_eyesupport.stl" scale="0.001 0.001 0.001"/>
+      </geometry>
+      <origin rpy="0 0 0" xyz="0 0 0"/>
+    </collision>
+</link>
   <link name="${side}_camera_link">
     <visual>
@@ -26,5 +32,11 @@
     </visual>
     <xacro:camera_inertial/>
-  </link>
+    <collision>
+      <geometry>
+        <mesh filename="package://inmoov_description/meshes/camera.stl" scale="0.001 0.001 0.001"/>
+      </geometry>
+      <origin rpy="0 0 0" xyz="0 0 0"/>
+    </collision>
+</link>
   <link name="${side}_eye_link">
     <visual>
@@ -36,5 +48,11 @@
     </visual>
     <xacro:eye_inertial/>
-  </link>
+    <collision>
+      <geometry>
+        <mesh filename="package://inmoov_description/meshes/eye.stl" scale="0.001 0.001 0.001"/>
+      </geometry>
+      <origin rpy="0 0 0" xyz="0 0 0"/>
+    </collision>
+</link>
   <link name="${side}_iris_link">
     <visual>
@@ -46,5 +64,11 @@
     </visual>
     <xacro:iris_inertial/>
-  </link>
+    <collision>
+      <geometry>
+        <mesh filename="package://inmoov_description/meshes/iris.stl" scale="0.001 0.001 0.001"/>
+      </geometry>
+      <origin rpy="0 0 0" xyz="0 0 0"/>
+    </collision>
+</link>
   <joint name="${side}_camera_joint" type="fixed">
     <origin rpy="0 0 0" xyz="-0.001 0 0"/>

File: inmoov_description/urdf/asmFace.urdf.xacro (robot description, xacro)
@@ -12,5 +12,11 @@
     </visual>
     <xacro:face_inertial/>
-  </link>
+    <collision>
+      <geometry>
+        <mesh filename="package://inmoov_description/meshes/face.stl" scale="0.001 0.001 0.001"/>
+      </geometry>
+      <origin rpy="0 0 0" xyz="0 0 0"/>
+    </collision>
+</link>
   <joint name="eyes_tilt_joint" type="revolute">
    <axis xyz="0 1 0"/>
@@ -29,5 +35,11 @@
     </visual>
     <xacro:eyesupport_inertial/>
-  </link>
+    <collision>
+      <geometry>
+        <mesh filename="package://inmoov_description/meshes/eyesupport.stl" scale="0.001 0.001 0.001"/>
+      </geometry>
+      <origin rpy="0 0 0" xyz="0 0 0"/>
+    </collision>
+</link>
 <xacro:asmEye side="r"/>
   <joint name="eyes_pan_joint" type="revolute">

File: inmoov_description/urdf/asmHand.urdf.xacro (robot description, xacro)
@@ -17,5 +17,11 @@
         <xacro:r_hand_inertial/>
       </xacro:if>
-    </link>
+    <collision>
+      <geometry>
+          <mesh filename="package://inmoov_description/meshes/${side}_hand.stl" scale="0.001 0.001 0.001"/>
+        </geometry>
+      <origin rpy="0 0 0" xyz="0 0 0"/>
+    </collision>
+</link>
     <link name="${side}_thumb1_link">
       <visual>
@@ -32,5 +38,11 @@
         <xacro:r_thumb5_1_inertial/>
       </xacro:if>
-    </link>
+    <collision>
+      <geometry>
+          <mesh filename="package://inmoov_description/meshes/${side}_thumb5_1.stl" scale="0.001 0.001 0.001"/>
+        </geometry>
+      <origin rpy="0 0 0" xyz="0 0 0"/>
+    </collision>
+</link>
     <link name="${side}_thumb2_link">
       <visual>
@@ -42,5 +54,11 @@
       </visual>
       <xacro:thumb5_2_inertial/>
-    </link>
+    <collision>
+      <geometry>
+          <mesh filename="package://inmoov_description/meshes/thumb5_2.stl" scale="0.001 0.001 0.001"/>
+        </geometry>
+      <origin rpy="0 0 0" xyz="0 0 0"/>
+    </collision>
+</link>
     <link name="${side}_thumb3_link">
       <visual>
@@ -52,5 +70,11 @@
       </visual>
       <xacro:thumb5_3_inertial/>
-    </link>
+    <collision>
+      <geometry>
+          <mesh filename="package://inmoov_description/meshes/thumb5_3.stl" scale="0.001 0.001 0.001"/>
+        </geometry>
+      <origin rpy="0 0 0" xyz="0 0 0"/>
+    </collision>
+</link>
     <link name="${side}_index1_link">
       <visual>
@@ -62,5 +86,11 @@
       </visual>
       <xacro:index3_1_inertial/>
-    </link>
+    <collision>
+      <geometry>
+          <mesh filename="package://inmoov_description/meshes/index3_1.stl" scale="0.001 0.001 0.001"/>
+        </geometry>
+      <origin rpy="0 0 0" xyz="0 0 0"/>
+    </collision>
+</link>
     <link name="${side}_index2_link">
       <visual>
@@ -72,5 +102,11 @@
       </visual>
       <xacro:index3_2_inertial/>
-    </link>
+    <collision>
+      <geometry>
+          <mesh filename="package://inmoov_description/meshes/index3_2.stl" scale="0.001 0.001 0.001"/>
+        </geometry>
+      <origin rpy="0 0 0" xyz="0 0 0"/>
+    </collision>
+</link>
     <link name="${side}_index3_link">
       <visual>
@@ -82,5 +118,11 @@
       </visual>
       <xacro:index3_3_inertial/>
-    </link>
+    <collision>
+      <geometry>
+          <mesh filename="package://inmoov_description/meshes/index3_3.stl" scale="0.001 0.001 0.001"/>
+        </geometry>
+      <origin rpy="0 0 0" xyz="0 0 0"/>
+    </collision>
+</link>
     <link name="${side}_middle1_link">
       <visual>
@@ -92,5 +134,11 @@
       </visual>
       <xacro:middle3_1_inertial/>
-    </link>
+    <collision>
+      <geometry>
+          <mesh filename="package://inmoov_description/meshes/middle3_1.stl" scale="0.001 0.001 0.001"/>
+        </geometry>
+      <origin rpy="0 0 0" xyz="0 0 0"/>
+    </collision>
+</link>
     <link name="${side}_middle2_link">
       <visual>
@@ -102,5 +150,11 @@
       </visual>
       <xacro:middle3_2_inertial/>
-    </link>
+    <collision>
+      <geometry>
+          <mesh filename="package://inmoov_description/meshes/middle3_2.stl" scale="0.001 0.001 0.001"/>
+        </geometry>
+      <origin rpy="0 0 0" xyz="0 0 0"/>
+    </collision>
+</link>
     <link name="${side}_middle3_link">
       <visual>
@@ -112,5 +166,11 @@
       </visual>
       <xacro:middle3_3_inertial/>
-    </link>
+    <collision>
+      <geometry>
+          <mesh filename="package://inmoov_description/meshes/middle3_3.stl" scale="0.001 0.001 0.001"/>
+        </geometry>
+      <origin rpy="0 0 0" xyz="0 0 0"/>
+    </collision>
+</link>
     <link name="${side}_ring1_link">
       <visual>
@@ -127,5 +187,11 @@
         <xacro:r_ring3_1_inertial/>
       </xacro:if>
-    </link>
+    <collision>
+      <geometry>
+          <mesh filename="package://inmoov_description/meshes/${side}_ring3_1.stl" scale="0.001 0.001 0.001"/>
+        </geometry>
+      <origin rpy="0 0 0" xyz="0 0 0"/>
+    </collision>
+</link>
     <link name="${side}_ring2_link">
       <visual>
@@ -137,5 +203,11 @@
       </visual>
       <xacro:ring3_2_inertial/>
-    </link>
+    <collision>
+      <geometry>
+          <mesh filename="package://inmoov_description/meshes/ring3_2.stl" scale="0.001 0.001 0.001"/>
+        </geometry>
+      <origin rpy="0 0 0" xyz="0 0 0"/>
+    </collision>
+</link>
     <link name="${side}_ring3_link">
       <visual>
@@ -147,5 +219,11 @@
       </visual>
       <xacro:ring3_3_inertial/>
-    </link>
+    <collision>
+      <geometry>
+          <mesh filename="package://inmoov_description/meshes/ring3_3.stl" scale="0.001 0.001 0.001"/>
+        </geometry>
+      <origin rpy="0 0 0" xyz="0 0 0"/>
+    </collision>
+</link>
     <link name="${side}_ring4_link">
       <visual>
@@ -157,5 +235,11 @@
       </visual>
       <xacro:ring3_4_inertial/>
-    </link>
+    <collision>
+      <geometry>
+          <mesh filename="package://inmoov_description/meshes/ring3_4.stl" scale="0.001 0.001 0.001"/>
+        </geometry>
+      <origin rpy="0 0 0" xyz="0 0 0"/>
+    </collision>
+</link>
     <link name="${side}_pinky1_link">
       <visual>
@@ -172,5 +256,11 @@
         <xacro:r_pinky3_1_inertial/>
       </xacro:if>
-    </link>
+    <collision>
+      <geometry>
+          <mesh filename="package://inmoov_description/meshes/${side}_pinky3_1.stl" scale="0.001 0.001 0.001"/>
+        </geometry>
+      <origin rpy="0 0 0" xyz="0 0 0"/>
+    </collision>
+</link>
     <link name="${side}_pinky2_link">
       <visual>
@@ -182,5 +272,11 @@
       </visual>
       <xacro:pinky3_2_inertial/>
-    </link>
+    <collision>
+      <geometry>
+          <mesh filename="package://inmoov_description/meshes/pinky3_2.stl" scale="0.001 0.001 0.001"/>
+        </geometry>
+      <origin rpy="0 0 0" xyz="0 0 0"/>
+    </collision>
+</link>
     <link name="${side}_pinky3_link">
       <visual>
@@ -192,5 +288,11 @@
       </visual>
       <xacro:pinky3_3_inertial/>
-    </link>
+    <collision>
+      <geometry>
+          <mesh filename="package://inmoov_description/meshes/pinky3_3.stl" scale="0.001 0.001 0.001"/>
+        </geometry>
+      <origin rpy="0 0 0" xyz="0 0 0"/>
+    </collision>
+</link>
     <link name="${side}_pinky4_link">
       <visual>
@@ -202,5 +304,11 @@
       </visual>
       <xacro:pinky3_4_inertial/>
-    </link>
+    <collision>
+      <geometry>
+          <mesh filename="package://inmoov_description/meshes/pinky3_4.stl" scale="0.001 0.001 0.001"/>
+        </geometry>
+      <origin rpy="0 0 0" xyz="0 0 0"/>
+    </collision>
+</link>
     <joint name="${side}_thumb1_joint" type="revolute">
       <axis xyz="0 0 1"/>
@@ -433,5 +541,11 @@
         <xacro:r_cover_hand_inertial/>
       </xacro:if>
-    </link>
+    <collision>
+      <geometry>
+          <mesh filename="package://inmoov_description/meshes/${side}_cover_hand.stl" scale="0.001 0.001 0.001"/>
+        </geometry>
+      <origin rpy="0 0 0" xyz="0 0 0"/>
+    </collision>
+</link>
     <link name="${side}_cover_handring_link">
       <visual>
@@ -448,5 +562,11 @@
         <xacro:r_cover_handring_inertial/>
       </xacro:if>
-    </link>
+    <collision>
+      <geometry>
+          <mesh filename="package://inmoov_description/meshes/${side}_cover_handring.stl" scale="0.001 0.001 0.001"/>
+        </geometry>
+      <origin rpy="0 0 0" xyz="0 0 0"/>
+    </collision>
+</link>
     <link name="${side}_cover_handpinky_link">
       <visual>
@@ -463,5 +583,11 @@
         <xacro:r_cover_handpinky_inertial/>
       </xacro:if>
-    </link>
+    <collision>
+      <geometry>
+          <mesh filename="package://inmoov_description/meshes/${side}_cover_handpinky.stl" scale="0.001 0.001 0.001"/>
+        </geometry>
+      <origin rpy="0 0 0" xyz="0 0 0"/>
+    </collision>
+</link>
     <link name="${side}_cover_thumb_link">
       <visual>
@@ -478,5 +604,11 @@
         <xacro:r_cover_thumb_inertial/>
       </xacro:if>
-    </link>
+    <collision>
+      <geometry>
+          <mesh filename="package://inmoov_description/meshes/${side}_cover_thumb.stl" scale="0.001 0.001 0.001"/>
+        </geometry>
+      <origin rpy="0 0 0" xyz="0 0 0"/>
+    </collision>
+</link>
     <link name="${side}_cover_index_link">
       <visual>
@@ -493,5 +625,11 @@
         <xacro:r_cover_index_inertial/>
       </xacro:if>
-    </link>
+    <collision>
+      <geometry>
+          <mesh filename="package://inmoov_description/meshes/${side}_cover_index.stl" scale="0.001 0.001 0.001"/>
+        </geometry>
+      <origin rpy="0 0 0" xyz="0 0 0"/>
+    </collision>
+</link>
     <link name="${side}_cover_middle_link">
       <visual>
@@ -508,5 +646,11 @@
         <xacro:r_cover_middle_inertial/>
       </xacro:if>
-    </link>
+    <collision>
+      <geometry>
+          <mesh filename="package://inmoov_description/meshes/${side}_cover_middle.stl" scale="0.001 0.001 0.001"/>
+        </geometry>
+      <origin rpy="0 0 0" xyz="0 0 0"/>
+    </collision>
+</link>
     <link name="${side}_cover_ring_link">
       <visual>
@@ -523,5 +667,11 @@
         <xacro:r_cover_ring_inertial/>
       </xacro:if>
-    </link>
+    <collision>
+      <geometry>
+          <mesh filename="package://inmoov_description/meshes/${side}_cover_ring.stl" scale="0.001 0.001 0.001"/>
+        </geometry>
+      <origin rpy="0 0 0" xyz="0 0 0"/>
+    </collision>
+</link>
     <link name="${side}_cover_pinky_link">
       <visual>
@@ -538,5 +688,11 @@
         <xacro:r_cover_pinky_inertial/>
       </xacro:if>
-    </link>
+    <collision>
+      <geometry>
+          <mesh filename="package://inmoov_description/meshes/${side}_cover_pinky.stl" scale="0.001 0.001 0.001"/>
+        </geometry>
+      <origin rpy="0 0 0" xyz="0 0 0"/>
+    </collision>
+</link>
     <joint name="${side}_handcover_joint" type="fixed">
       <origin rpy="0 0 0" xyz="0.009 ${flip * 0.0192} -0.0977"/>

File: inmoov_description/urdf/asmHead.urdf.xacro (robot description, xacro)
@@ -11,5 +11,11 @@
     </visual>
     <xacro:head_base_inertial/>
-  </link>
+    <collision>
+      <geometry>
+        <mesh filename="package://inmoov_description/meshes/head_base.stl" scale="0.001 0.001 0.001"/>
+      </geometry>
+      <origin rpy="0 0 0" xyz="0 0 0"/>
+    </collision>
+</link>
   <link name="head_link">
     <visual>
@@ -21,5 +27,11 @@
     </visual>
     <xacro:head_inertial/>
-  </link>
+    <collision>
+      <geometry>
+        <mesh filename="package://inmoov_description/meshes/head.stl" scale="0.001 0.001 0.001"/>
+      </geometry>
+      <origin rpy="0 0 0" xyz="0 0 0"/>
+    </collision>
+</link>
   <link name="jaw_link">
     <visual>
@@ -31,5 +43,11 @@
     </visual>
     <xacro:jaw_inertial/>
-  </link>
+    <collision>
+      <geometry>
+        <mesh filename="package://inmoov_description/meshes/jaw.stl" scale="0.001 0.001 0.001"/>
+      </geometry>
+      <origin rpy="0 0 0" xyz="0 0 0"/>
+    </collision>
+</link>
   <link name="skull_link">
     <visual>
@@ -41,5 +59,11 @@
     </visual>
     <xacro:skull_inertial/>
-  </link>
+    <collision>
+      <geometry>
+        <mesh filename="package://inmoov_description/meshes/skull.stl" scale="0.001 0.001 0.001"/>
+      </geometry>
+      <origin rpy="0 0 0" xyz="0 0 0"/>
+    </collision>
+</link>
   <link name="left_ear_link">
     <visual>
@@ -51,5 +75,11 @@
     </visual>
     <xacro:earleftv1_inertial/>
-  </link>
+    <collision>
+      <geometry>
+        <mesh filename="package://inmoov_description/meshes/earleftv1.stl" scale="0.001 0.001 0.001"/>
+      </geometry>
+      <origin rpy="0 0 0" xyz="0 0 0"/>
+    </collision>
+</link>
   <link name="right_ear_link">
     <visual>
@@ -61,5 +91,11 @@
     </visual>
     <xacro:earrightv1_inertial/>
-  </link>
+    <collision>
+      <geometry>
+        <mesh filename="package://inmoov_description/meshes/earrightv1.stl" scale="0.001 0.001 0.001"/>
+      </geometry>
+      <origin rpy="0 0 0" xyz="0 0 0"/>
+    </collision>
+</link>
   <joint name="head_pan_joint" type="revolute">
    <axis xyz="0 0 1"/>

File: inmoov_description/urdf/asmTorso.urdf.xacro (robot description, xacro)
@@ -11,5 +11,11 @@
     </visual>
     <xacro:mid_stomach_inertial/>
-  </link>
+    <collision>
+      <geometry>
+        <mesh filename="package://inmoov_description/meshes/mid_stomach.stl" scale="0.001 0.001 0.001"/>
+      </geometry>
+      <origin rpy="0 0 0" xyz="0 0 1.152"/>
+    </collision>
+</link>
   <link name="disk_link">
     <visual>
@@ -21,5 +27,11 @@
     </visual>
     <xacro:disk_inertial/>
-  </link>
+    <collision>
+      <geometry>
+        <mesh filename="package://inmoov_description/meshes/disk.stl" scale="0.001 0.001 0.001"/>
+      </geometry>
+      <origin rpy="0 0 0" xyz="0 0 0"/>
+    </collision>
+</link>
   <link name="top_stomach_link">
     <visual>
@@ -31,5 +43,11 @@
     </visual>
     <xacro:top_stomach_inertial/>
-  </link>
+    <collision>
+      <geometry>
+        <mesh filename="package://inmoov_description/meshes/top_stomach.stl" scale="0.001 0.001 0.001"/>
+      </geometry>
+      <origin rpy="0 0 0" xyz="0 0 0"/>
+    </collision>
+</link>
   <link name="torso_link">
     <visual>
@@ -41,5 +59,11 @@
     </visual>
     <xacro:torso_inertial/>
-  </link>
+    <collision>
+      <geometry>
+        <mesh filename="package://inmoov_description/meshes/torso.stl" scale="0.001 0.001 0.001"/>
+      </geometry>
+      <origin rpy="0 0 0" xyz="0 0 0"/>
+    </collision>
+</link>
   <link name="kinect2_link">
     <visual>
@@ -51,5 +75,11 @@
     </visual>
     <xacro:kinectone_inertial/>
-  </link>
+    <collision>
+      <geometry>
+        <mesh filename="package://inmoov_description/meshes/kinectone.stl" scale="0.001 0.001 0.001"/>
+      </geometry>
+      <origin rpy="1.57 0 0" xyz="0 0 0"/>
+    </collision>
+</link>
   <link name="kinect2_ir_optical_frame">
     <visual>
@@ -61,5 +91,11 @@
     </visual>
     <xacro:kinectone_inertial/>
-  </link>
+    <collision>
+      <geometry>
+        <mesh filename="package://inmoov_description/meshes/kinectone.stl" scale="0.001 0.001 0.001"/>
+      </geometry>
+      <origin rpy="1.57 0 0" xyz="0 0 0"/>
+    </collision>
+</link>
   <link name="kinect2_rgb_optical_frame">
     <visual>
@@ -71,5 +107,11 @@
     </visual>
     <xacro:kinectone_inertial/>
-  </link>
+    <collision>
+      <geometry>
+        <mesh filename="package://inmoov_description/meshes/kinectone.stl" scale="0.001 0.001 0.001"/>
+      </geometry>
+      <origin rpy="1.57 0 0" xyz="0 0 0"/>
+    </collision>
+</link>
   <link name="chestplate_link">
     <visual>
@@ -81,5 +123,11 @@
     </visual>
     <xacro:chest_inertial/>
-  </link>
+    <collision>
+      <geometry>
+        <mesh filename="package://inmoov_description/meshes/chest.stl" scale="0.001 0.001 0.001"/>
+      </geometry>
+      <origin rpy="0 0 0" xyz="0 0 0"/>
+    </collision>
+</link>
   <joint name="waist_pan_joint" type="revolute">
    <axis xyz="0 0 1"/>
