Commit message: Updated mass and effort

File: inmoov_description/robots/inmoov.urdf.xacro (robot description, xacro)
@@ -78,5 +78,5 @@
   <joint name="head_roll_joint" type="revolute">
    <axis xyz="1 0 0"/>
-   <limit effort="1000.0" lower="${head_roll_joint_lower}" upper="${head_roll_joint_upper}" velocity="${head_roll_joint_velocity}" />
+   <limit effort="10000.0" lower="${head_roll_joint_lower}" upper="${head_roll_joint_upper}" velocity="${head_roll_joint_velocity}" />
    <origin rpy="0 0 3.1415" xyz="-0.0315  -0.001 0.4551"/>
    <parent link="torso_link"/>
@@ -85,5 +85,5 @@
   <joint name="head_tilt_joint" type="revolute">
    <axis xyz="0 1 0"/>
-   <limit effort="1000.0" lower="${head_tilt_joint_lower}" upper="${head_tilt_joint_upper}" velocity="${head_tilt_joint_velocity}" />
+   <limit effort="10000.0" lower="${head_tilt_joint_lower}" upper="${head_tilt_joint_upper}" velocity="${head_tilt_joint_velocity}" />
    <origin rpy="0 0 3.1415" xyz="0 0 0"/>
    <parent link="head_tilt_link"/>
@@ -100,5 +100,5 @@
   <joint name="r_shoulder_out_joint" type="revolute">
    <axis xyz="1 0 0"/>
-   <limit effort="1000.0" lower="${r_shoulder_out_joint_lower}" upper="${r_shoulder_out_joint_upper}" velocity="${r_shoulder_out_joint_velocity}" />
+   <limit effort="10000.0" lower="${r_shoulder_out_joint_lower}" upper="${r_shoulder_out_joint_upper}" velocity="${r_shoulder_out_joint_velocity}" />
    <origin rpy="0 0 0" xyz="0 -0.143 0.298"/>
    <parent link="torso_link"/>
@@ -108,5 +108,5 @@
   <joint name="r_wrist_roll_joint" type="revolute">
    <axis xyz="0 0 1"/>
-   <limit effort="1000.0" lower="${r_wrist_roll_joint_lower}" upper="${r_wrist_roll_joint_upper}" velocity="${r_wrist_roll_joint_velocity}" />
+   <limit effort="10000.0" lower="${r_wrist_roll_joint_lower}" upper="${r_wrist_roll_joint_upper}" velocity="${r_wrist_roll_joint_velocity}" />
    <origin rpy="0 0 0" xyz="-0.0144 0.01  -0.2885"/>
    <parent link="r_forearm_link"/>
@@ -116,5 +116,5 @@
   <joint name="l_shoulder_out_joint" type="revolute">
    <axis xyz="1 0 0"/>
-   <limit effort="1000.0" lower="${l_shoulder_out_joint_lower}" upper="${l_shoulder_out_joint_upper}" velocity="${l_shoulder_out_joint_velocity}" />
+   <limit effort="10000.0" lower="${l_shoulder_out_joint_lower}" upper="${l_shoulder_out_joint_upper}" velocity="${l_shoulder_out_joint_velocity}" />
    <origin rpy="0 0 0" xyz="0 0.143 0.298"/>
    <parent link="torso_link"/>
@@ -124,5 +124,5 @@
   <joint name="l_wrist_roll_joint" type="revolute">
    <axis xyz="0 0 1"/>
-   <limit effort="1000.0" lower="${l_wrist_roll_joint_lower}" upper="${l_wrist_roll_joint_upper}" velocity="${l_wrist_roll_joint_velocity}" />
+   <limit effort="10000.0" lower="${l_wrist_roll_joint_lower}" upper="${l_wrist_roll_joint_upper}" velocity="${l_wrist_roll_joint_velocity}" />
    <origin rpy="0 0 0" xyz="-0.0144 -0.01  -0.2885"/>
    <parent link="l_forearm_link"/>

File: inmoov_description/robots/inmoov_face.urdf.xacro (robot description, xacro)
@@ -18,5 +18,5 @@
   <joint name="base_to_face" type="revolute">
    <axis xyz="0 0 1"/>
-<limit effort="1000.0" lower="-3.14" upper="0" velocity="0.5"/>
+<limit effort="10000.0" lower="-3.14" upper="0" velocity="0.5"/>
 <origin rpy="0 0 0" xyz="0 0 0"/>
     <parent link="base_link"/>

File: inmoov_description/robots/inmoov_head.urdf.xacro (robot description, xacro)
@@ -21,5 +21,5 @@
   <joint name="base_to_base" type="revolute">
    <axis xyz="0 0 1"/>
-   <limit effort="1000.0" lower="-3.14" upper="0" velocity="0.5"/>
+   <limit effort="10000.0" lower="-3.14" upper="0" velocity="0.5"/>
    <origin rpy="0 0 0" xyz="0 0 0"/>
    <parent link="base_link"/>

File: inmoov_description/robots/inmoov_right_hand.urdf.xacro (robot description, xacro)
@@ -19,5 +19,5 @@
   <joint name="base_to_hand_joint" type="revolute">
    <axis xyz="0 0 1"/>
-<limit effort="1000.0" lower="-3.14" upper="0" velocity="0.5"/>
+<limit effort="10000.0" lower="-3.14" upper="0" velocity="0.5"/>
 <origin rpy="0 0 0" xyz="0 0 0"/>
     <parent link="base_link"/>

File: inmoov_description/urdf/asmArm.urdf.xacro (robot description, xacro)
@@ -100,8 +100,8 @@
     <axis xyz="0 1 0"/>
     <xacro:if value="${side == 'l'}">
-      <limit effort="1000.0" lower="${l_shoulder_lift_joint_lower}" upper="${l_shoulder_lift_joint_upper}" velocity="${l_shoulder_lift_joint_velocity}" />
+      <limit effort="10000.0" lower="${l_shoulder_lift_joint_lower}" upper="${l_shoulder_lift_joint_upper}" velocity="${l_shoulder_lift_joint_velocity}" />
     </xacro:if>
     <xacro:if value="${side == 'r'}">
-      <limit effort="1000.0" lower="${r_shoulder_lift_joint_lower}" upper="${r_shoulder_lift_joint_upper}" velocity="${r_shoulder_lift_joint_velocity}" />
+      <limit effort="10000.0" lower="${r_shoulder_lift_joint_lower}" upper="${r_shoulder_lift_joint_upper}" velocity="${r_shoulder_lift_joint_velocity}" />
     </xacro:if>
     <origin rpy="0 0 0" xyz="0 ${flip * -0.012} -0.04"/>
@@ -112,8 +112,8 @@
     <axis xyz="0 0 1"/>
     <xacro:if value="${side == 'l'}">
-      <limit effort="1000.0" lower="${l_upper_arm_roll_joint_lower}" upper="${l_upper_arm_roll_joint_upper}" velocity="${l_upper_arm_roll_joint_velocity}" />
+      <limit effort="10000.0" lower="${l_upper_arm_roll_joint_lower}" upper="${l_upper_arm_roll_joint_upper}" velocity="${l_upper_arm_roll_joint_velocity}" />
     </xacro:if>
     <xacro:if value="${side == 'r'}">
-      <limit effort="1000.0" lower="${r_upper_arm_roll_joint_lower}" upper="${r_upper_arm_roll_joint_upper}" velocity="${r_upper_arm_roll_joint_velocity}" />
+      <limit effort="10000.0" lower="${r_upper_arm_roll_joint_lower}" upper="${r_upper_arm_roll_joint_upper}" velocity="${r_upper_arm_roll_joint_velocity}" />
     </xacro:if>
     <origin rpy="0 0 0" xyz="0 ${flip * -0.066} -0.060"/>
@@ -124,8 +124,8 @@
     <axis xyz="0 1 0"/>
     <xacro:if value="${side == 'l'}">
-      <limit effort="1000.0" lower="${l_elbow_flex_joint_lower}" upper="${l_elbow_flex_joint_upper}" velocity="${l_elbow_flex_joint_velocity}" />
+      <limit effort="10000.0" lower="${l_elbow_flex_joint_lower}" upper="${l_elbow_flex_joint_upper}" velocity="${l_elbow_flex_joint_velocity}" />
     </xacro:if>
     <xacro:if value="${side == 'r'}">
-      <limit effort="1000.0" lower="${r_elbow_flex_joint_lower}" upper="${r_elbow_flex_joint_upper}" velocity="${r_elbow_flex_joint_velocity}" />
+      <limit effort="10000.0" lower="${r_elbow_flex_joint_lower}" upper="${r_elbow_flex_joint_upper}" velocity="${r_elbow_flex_joint_velocity}" />
     </xacro:if>
     <origin rpy="0 0 0" xyz="-0.0278 0 -0.2235"/>

File: inmoov_description/urdf/asmFace.urdf.xacro (robot description, xacro)
@@ -21,5 +21,5 @@
   <joint name="eyes_tilt_joint" type="revolute">
    <axis xyz="0 1 0"/>
-   <limit effort="1000.0" lower="${eyes_tilt_joint_lower}" upper="${eyes_tilt_joint_upper}" velocity="${eyes_tilt_joint_velocity}" />
+   <limit effort="10000.0" lower="${eyes_tilt_joint_lower}" upper="${eyes_tilt_joint_upper}" velocity="${eyes_tilt_joint_velocity}" />
    <origin rpy="0 0 0" xyz="0 0 0"/>
    <parent link="face_link"/>
@@ -45,5 +45,5 @@
   <joint name="eyes_pan_joint" type="revolute">
    <axis xyz="0 0 1"/>
-    <limit effort="1000.0" lower="${eyes_pan_joint_lower}" upper="${eyes_pan_joint_upper}" velocity="${eyes_pan_joint_velocity}" />
+    <limit effort="10000.0" lower="${eyes_pan_joint_lower}" upper="${eyes_pan_joint_upper}" velocity="${eyes_pan_joint_velocity}" />
    <origin rpy="0 0 0" xyz="0 0.033 -0.0036"/>
    <parent link="eyesupport_link"/>
@@ -53,5 +53,5 @@
   <joint name="l_eye_pan_joint" type="revolute">
    <axis xyz="0 0 1"/>
-   <limit effort="1000.0" lower="${eyes_pan_joint_lower}" upper="${eyes_pan_joint_upper}" velocity="${eyes_pan_joint_velocity}" />
+   <limit effort="10000.0" lower="${eyes_pan_joint_lower}" upper="${eyes_pan_joint_upper}" velocity="${eyes_pan_joint_velocity}" />
    <mimic joint="eyes_pan_joint" multiplier="1" offset="0"/>
    <origin rpy="0 0 0" xyz="0 -0.033 -0.0036"/>

File: inmoov_description/urdf/asmHand.urdf.xacro (robot description, xacro)
@@ -314,8 +314,8 @@
       <axis xyz="0 0 1"/>
         <xacro:if value="${side == 'l'}">
-          <limit effort="1000.0" lower="${l_thumb_joint_lower}" upper="${l_thumb_joint_upper}" velocity="${l_thumb_joint_velocity}" />
-        </xacro:if>
-        <xacro:if value="${side == 'r'}">
-          <limit effort="1000.0" lower="${r_thumb_joint_lower}" upper="${r_thumb_joint_upper}" velocity="${r_thumb_joint_velocity}" />
+          <limit effort="10000.0" lower="${l_thumb_joint_lower}" upper="${l_thumb_joint_upper}" velocity="${l_thumb_joint_velocity}" />
+        </xacro:if>
+        <xacro:if value="${side == 'r'}">
+          <limit effort="10000.0" lower="${r_thumb_joint_lower}" upper="${r_thumb_joint_upper}" velocity="${r_thumb_joint_velocity}" />
         </xacro:if>
       <origin rpy="${flip * 0.1} 0 0" xyz="0 ${flip * 0.029} -0.0577"/>
@@ -327,8 +327,8 @@
       <axis xyz="0 1 0"/>
         <xacro:if value="${side == 'l'}">
-          <limit effort="1000.0" lower="${l_thumb_joint_lower}" upper="${l_thumb_joint_upper}" velocity="${l_thumb_joint_velocity}" />
-        </xacro:if>
-        <xacro:if value="${side == 'r'}">
-          <limit effort="1000.0" lower="${r_thumb_joint_lower}" upper="${r_thumb_joint_upper}" velocity="${r_thumb_joint_velocity}" />
+          <limit effort="10000.0" lower="${l_thumb_joint_lower}" upper="${l_thumb_joint_upper}" velocity="${l_thumb_joint_velocity}" />
+        </xacro:if>
+        <xacro:if value="${side == 'r'}">
+          <limit effort="10000.0" lower="${r_thumb_joint_lower}" upper="${r_thumb_joint_upper}" velocity="${r_thumb_joint_velocity}" />
         </xacro:if>
       <origin rpy="${flip * 0.825} -0.1 ${flip * 0.3}" xyz="-0.00052 ${flip * 0.02725}  -0.013"/>
@@ -339,8 +339,8 @@
       <axis xyz="0 1 0"/>
         <xacro:if value="${side == 'l'}">
-          <limit effort="1000.0" lower="${l_thumb_joint_lower}" upper="${l_thumb_joint_upper}" velocity="${l_thumb_joint_velocity}" />
-        </xacro:if>
-        <xacro:if value="${side == 'r'}">
-          <limit effort="1000.0" lower="${r_thumb_joint_lower}" upper="${r_thumb_joint_upper}" velocity="${r_thumb_joint_velocity}" />
+          <limit effort="10000.0" lower="${l_thumb_joint_lower}" upper="${l_thumb_joint_upper}" velocity="${l_thumb_joint_velocity}" />
+        </xacro:if>
+        <xacro:if value="${side == 'r'}">
+          <limit effort="10000.0" lower="${r_thumb_joint_lower}" upper="${r_thumb_joint_upper}" velocity="${r_thumb_joint_velocity}" />
         </xacro:if>
       <origin rpy="0 0 0" xyz="0 0 -0.035"/>
@@ -352,8 +352,8 @@
       <axis xyz="0 1 0"/>
         <xacro:if value="${side == 'l'}">
-          <limit effort="1000.0" lower="${l_index_joint_lower}" upper="${l_index_joint_upper}" velocity="${l_index_joint_velocity}" />
-        </xacro:if>
-        <xacro:if value="${side == 'r'}">
-          <limit effort="1000.0" lower="${r_index_joint_lower}" upper="${r_index_joint_upper}" velocity="${r_index_joint_velocity}" />
+          <limit effort="10000.0" lower="${l_index_joint_lower}" upper="${l_index_joint_upper}" velocity="${l_index_joint_velocity}" />
+        </xacro:if>
+        <xacro:if value="${side == 'r'}">
+          <limit effort="10000.0" lower="${r_index_joint_lower}" upper="${r_index_joint_upper}" velocity="${r_index_joint_velocity}" />
         </xacro:if>
       <origin rpy="${flip * 0.1} 0 0" xyz="-0.0015 ${flip * 0.0342}  -0.119"/>
@@ -365,8 +365,8 @@
       <axis xyz="0 1 0"/>
         <xacro:if value="${side == 'l'}">
-          <limit effort="1000.0" lower="${l_index_joint_lower}" upper="${l_index_joint_upper}" velocity="${l_index_joint_velocity}" />
-        </xacro:if>
-        <xacro:if value="${side == 'r'}">
-          <limit effort="1000.0" lower="${r_index_joint_lower}" upper="${r_index_joint_upper}" velocity="${r_index_joint_velocity}" />
+          <limit effort="10000.0" lower="${l_index_joint_lower}" upper="${l_index_joint_upper}" velocity="${l_index_joint_velocity}" />
+        </xacro:if>
+        <xacro:if value="${side == 'r'}">
+          <limit effort="10000.0" lower="${r_index_joint_lower}" upper="${r_index_joint_upper}" velocity="${r_index_joint_velocity}" />
         </xacro:if>
       <origin rpy="0 0 0" xyz="0 0.001 -0.03595"/>
@@ -377,8 +377,8 @@
       <axis xyz="0 1 0"/>
         <xacro:if value="${side == 'l'}">
-          <limit effort="1000.0" lower="${l_index_joint_lower}" upper="${l_index_joint_upper}" velocity="${l_index_joint_velocity}" />
-        </xacro:if>
-        <xacro:if value="${side == 'r'}">
-          <limit effort="1000.0" lower="${r_index_joint_lower}" upper="${r_index_joint_upper}" velocity="${r_index_joint_velocity}" />
+          <limit effort="10000.0" lower="${l_index_joint_lower}" upper="${l_index_joint_upper}" velocity="${l_index_joint_velocity}" />
+        </xacro:if>
+        <xacro:if value="${side == 'r'}">
+          <limit effort="10000.0" lower="${r_index_joint_lower}" upper="${r_index_joint_upper}" velocity="${r_index_joint_velocity}" />
         </xacro:if>
       <origin rpy="0 0 0" xyz="0 0 -0.024"/>
@@ -390,8 +390,8 @@
       <axis xyz="0 1 0"/>
         <xacro:if value="${side == 'l'}">
-          <limit effort="1000.0" lower="${l_middle_joint_lower}" upper="${l_middle_joint_upper}" velocity="${l_middle_joint_velocity}" />
-        </xacro:if>
-        <xacro:if value="${side == 'r'}">
-          <limit effort="1000.0" lower="${r_middle_joint_lower}" upper="${r_middle_joint_upper}" velocity="${r_middle_joint_velocity}" />
+          <limit effort="10000.0" lower="${l_middle_joint_lower}" upper="${l_middle_joint_upper}" velocity="${l_middle_joint_velocity}" />
+        </xacro:if>
+        <xacro:if value="${side == 'r'}">
+          <limit effort="10000.0" lower="${r_middle_joint_lower}" upper="${r_middle_joint_upper}" velocity="${r_middle_joint_velocity}" />
         </xacro:if>
       <origin rpy="0 0 0" xyz="-0.00175 ${flip * 0.007}  -0.12325"/>
@@ -403,8 +403,8 @@
       <axis xyz="0 1 0"/>
         <xacro:if value="${side == 'l'}">
-          <limit effort="1000.0" lower="${l_middle_joint_lower}" upper="${l_middle_joint_upper}" velocity="${l_middle_joint_velocity}" />
-        </xacro:if>
-        <xacro:if value="${side == 'r'}">
-          <limit effort="1000.0" lower="${r_middle_joint_lower}" upper="${r_middle_joint_upper}" velocity="${r_middle_joint_velocity}" />
+          <limit effort="10000.0" lower="${l_middle_joint_lower}" upper="${l_middle_joint_upper}" velocity="${l_middle_joint_velocity}" />
+        </xacro:if>
+        <xacro:if value="${side == 'r'}">
+          <limit effort="10000.0" lower="${r_middle_joint_lower}" upper="${r_middle_joint_upper}" velocity="${r_middle_joint_velocity}" />
         </xacro:if>
       <origin rpy="0 0 0" xyz="0 0.000 -0.0389"/>
@@ -415,8 +415,8 @@
       <axis xyz="0 1 0"/>
         <xacro:if value="${side == 'l'}">
-          <limit effort="1000.0" lower="${l_middle_joint_lower}" upper="${l_middle_joint_upper}" velocity="${l_middle_joint_velocity}" />
-        </xacro:if>
-        <xacro:if value="${side == 'r'}">
-          <limit effort="1000.0" lower="${r_middle_joint_lower}" upper="${r_middle_joint_upper}" velocity="${r_middle_joint_velocity}" />
+          <limit effort="10000.0" lower="${l_middle_joint_lower}" upper="${l_middle_joint_upper}" velocity="${l_middle_joint_velocity}" />
+        </xacro:if>
+        <xacro:if value="${side == 'r'}">
+          <limit effort="10000.0" lower="${r_middle_joint_lower}" upper="${r_middle_joint_upper}" velocity="${r_middle_joint_velocity}" />
         </xacro:if>
       <origin rpy="0 0 0" xyz="0 0.0005 -0.0259"/>
@@ -428,8 +428,8 @@
       <axis xyz="0 0 1"/>
         <xacro:if value="${side == 'l'}">
-          <limit effort="1000.0" lower="${l_ring_joint_lower}" upper="${l_ring_joint_upper}" velocity="${l_ring_joint_velocity}" />
-        </xacro:if>
-        <xacro:if value="${side == 'r'}">
-          <limit effort="1000.0" lower="${r_ring_joint_lower}" upper="${r_ring_joint_upper}" velocity="${r_ring_joint_velocity}" />
+          <limit effort="10000.0" lower="${l_ring_joint_lower}" upper="${l_ring_joint_upper}" velocity="${l_ring_joint_velocity}" />
+        </xacro:if>
+        <xacro:if value="${side == 'r'}">
+          <limit effort="10000.0" lower="${r_ring_joint_lower}" upper="${r_ring_joint_upper}" velocity="${r_ring_joint_velocity}" />
         </xacro:if>
       <origin rpy="${flip * 0.7} 0 0" xyz="0 ${flip * -0.00705} -0.0794"/>
@@ -441,8 +441,8 @@
       <axis xyz="0 1 0"/>
         <xacro:if value="${side == 'l'}">
-          <limit effort="1000.0" lower="${l_ring_joint_lower}" upper="${l_ring_joint_upper}" velocity="${l_ring_joint_velocity}" />
-        </xacro:if>
-        <xacro:if value="${side == 'r'}">
-          <limit effort="1000.0" lower="${r_ring_joint_lower}" upper="${r_ring_joint_upper}" velocity="${r_ring_joint_velocity}" />
+          <limit effort="10000.0" lower="${l_ring_joint_lower}" upper="${l_ring_joint_upper}" velocity="${l_ring_joint_velocity}" />
+        </xacro:if>
+        <xacro:if value="${side == 'r'}">
+          <limit effort="10000.0" lower="${r_ring_joint_lower}" upper="${r_ring_joint_upper}" velocity="${r_ring_joint_velocity}" />
         </xacro:if>
       <origin rpy="${flip * -0.7775} 0 0" xyz="0.00126 ${flip * -0.0351} -0.0166"/>
@@ -453,8 +453,8 @@
       <axis xyz="0 1 0"/>
         <xacro:if value="${side == 'l'}">
-          <limit effort="1000.0" lower="${l_ring_joint_lower}" upper="${l_ring_joint_upper}" velocity="${l_ring_joint_velocity}" />
-        </xacro:if>
-        <xacro:if value="${side == 'r'}">
-          <limit effort="1000.0" lower="${r_ring_joint_lower}" upper="${r_ring_joint_upper}" velocity="${r_ring_joint_velocity}" />
+          <limit effort="10000.0" lower="${l_ring_joint_lower}" upper="${l_ring_joint_upper}" velocity="${l_ring_joint_velocity}" />
+        </xacro:if>
+        <xacro:if value="${side == 'r'}">
+          <limit effort="10000.0" lower="${r_ring_joint_lower}" upper="${r_ring_joint_upper}" velocity="${r_ring_joint_velocity}" />
         </xacro:if>
       <origin rpy="0 0 0" xyz="0 0.0005 -0.0345"/>
@@ -466,8 +466,8 @@
       <axis xyz="0 1 0"/>
         <xacro:if value="${side == 'l'}">
-          <limit effort="1000.0" lower="${l_ring_joint_lower}" upper="${l_ring_joint_upper}" velocity="${l_ring_joint_velocity}" />
-        </xacro:if>
-        <xacro:if value="${side == 'r'}">
-          <limit effort="1000.0" lower="${r_ring_joint_lower}" upper="${r_ring_joint_upper}" velocity="${r_ring_joint_velocity}" />
+          <limit effort="10000.0" lower="${l_ring_joint_lower}" upper="${l_ring_joint_upper}" velocity="${l_ring_joint_velocity}" />
+        </xacro:if>
+        <xacro:if value="${side == 'r'}">
+          <limit effort="10000.0" lower="${r_ring_joint_lower}" upper="${r_ring_joint_upper}" velocity="${r_ring_joint_velocity}" />
         </xacro:if>
       <origin rpy="0 0 0" xyz="0 0.0004 -0.0229"/>
@@ -479,8 +479,8 @@
       <axis xyz="0 0 1"/>
         <xacro:if value="${side == 'l'}">
-          <limit effort="1000.0" lower="${l_pinky_joint_lower}" upper="${l_pinky_joint_upper}" velocity="${l_pinky_joint_velocity}" />
-        </xacro:if>
-        <xacro:if value="${side == 'r'}">
-          <limit effort="1000.0" lower="${r_pinky_joint_lower}" upper="${r_pinky_joint_upper}" velocity="${r_pinky_joint_velocity}" />
+          <limit effort="10000.0" lower="${l_pinky_joint_lower}" upper="${l_pinky_joint_upper}" velocity="${l_pinky_joint_velocity}" />
+        </xacro:if>
+        <xacro:if value="${side == 'r'}">
+          <limit effort="10000.0" lower="${r_pinky_joint_lower}" upper="${r_pinky_joint_upper}" velocity="${r_pinky_joint_velocity}" />
         </xacro:if>
       <origin rpy="${flip * 0.7} 0 0" xyz="0 ${flip * -0.0270} -0.0555"/>
@@ -492,8 +492,8 @@
       <axis xyz="0 1 0"/>
         <xacro:if value="${side == 'l'}">
-          <limit effort="1000.0" lower="${l_pinky_joint_lower}" upper="${l_pinky_joint_upper}" velocity="${l_pinky_joint_velocity}" />
-        </xacro:if>
-        <xacro:if value="${side == 'r'}">
-          <limit effort="1000.0" lower="${r_pinky_joint_lower}" upper="${r_pinky_joint_upper}" velocity="${r_pinky_joint_velocity}" />
+          <limit effort="10000.0" lower="${l_pinky_joint_lower}" upper="${l_pinky_joint_upper}" velocity="${l_pinky_joint_velocity}" />
+        </xacro:if>
+        <xacro:if value="${side == 'r'}">
+          <limit effort="10000.0" lower="${r_pinky_joint_lower}" upper="${r_pinky_joint_upper}" velocity="${r_pinky_joint_velocity}" />
         </xacro:if>
       <origin rpy="${flip * -0.93} 0 0" xyz="0 ${flip * -0.046} -0.0228"/>
@@ -504,8 +504,8 @@
       <axis xyz="0 1 0"/>
         <xacro:if value="${side == 'l'}">
-          <limit effort="1000.0" lower="${l_pinky_joint_lower}" upper="${l_pinky_joint_upper}" velocity="${l_pinky_joint_velocity}" />
-        </xacro:if>
-        <xacro:if value="${side == 'r'}">
-          <limit effort="1000.0" lower="${r_pinky_joint_lower}" upper="${r_pinky_joint_upper}" velocity="${r_pinky_joint_velocity}" />
+          <limit effort="10000.0" lower="${l_pinky_joint_lower}" upper="${l_pinky_joint_upper}" velocity="${l_pinky_joint_velocity}" />
+        </xacro:if>
+        <xacro:if value="${side == 'r'}">
+          <limit effort="10000.0" lower="${r_pinky_joint_lower}" upper="${r_pinky_joint_upper}" velocity="${r_pinky_joint_velocity}" />
         </xacro:if>
       <origin rpy="0 0 0" xyz="0 0.0005 -0.031"/>
@@ -517,8 +517,8 @@
       <axis xyz="0 1 0"/>
         <xacro:if value="${side == 'l'}">
-          <limit effort="1000.0" lower="${l_pinky_joint_lower}" upper="${l_pinky_joint_upper}" velocity="${l_pinky_joint_velocity}" />
-        </xacro:if>
-        <xacro:if value="${side == 'r'}">
-          <limit effort="1000.0" lower="${r_pinky_joint_lower}" upper="${r_pinky_joint_upper}" velocity="${r_pinky_joint_velocity}" />
+          <limit effort="10000.0" lower="${l_pinky_joint_lower}" upper="${l_pinky_joint_upper}" velocity="${l_pinky_joint_velocity}" />
+        </xacro:if>
+        <xacro:if value="${side == 'r'}">
+          <limit effort="10000.0" lower="${r_pinky_joint_lower}" upper="${r_pinky_joint_upper}" velocity="${r_pinky_joint_velocity}" />
         </xacro:if>
       <origin rpy="0 0 0" xyz="0 0.0004 -0.0208"/>
