Commit message: Updated mass and effort

File: inmoov_description/urdf/asmHead.urdf.xacro (robot description, xacro)
@@ -100,5 +100,5 @@
   <joint name="head_pan_joint" type="revolute">
    <axis xyz="0 0 1"/>
-   <limit effort="1000.0" lower="${head_pan_joint_lower}" upper="${head_pan_joint_upper}" velocity="${head_pan_joint_velocity}" />
+   <limit effort="10000.0" lower="${head_pan_joint_lower}" upper="${head_pan_joint_upper}" velocity="${head_pan_joint_velocity}" />
    <origin rpy="0 0 0" xyz="0 0 0.0245"/>
    <parent link="head_base_link"/>
@@ -107,5 +107,5 @@
   <joint name="jaw_joint" type="revolute">
    <axis xyz="0 1 0"/>
-   <limit effort="1000.0" lower="${jaw_joint_lower}" upper="${jaw_joint_upper}" velocity="${jaw_joint_velocity}" />
+   <limit effort="10000.0" lower="${jaw_joint_lower}" upper="${jaw_joint_upper}" velocity="${jaw_joint_velocity}" />
    <origin rpy="0 0.09 0" xyz="0.0375 0.0005 0.0437"/>
    <parent link="head_link"/>

File: inmoov_description/urdf/asmTorso.urdf.xacro (robot description, xacro)
@@ -132,5 +132,5 @@
   <joint name="waist_pan_joint" type="revolute">
    <axis xyz="0 0 1"/>
-   <limit effort="1000.0" lower="${waist_pan_joint_lower}" upper="${waist_pan_joint_upper}" velocity="${waist_pan_joint_velocity}" />
+   <limit effort="10000.0" lower="${waist_pan_joint_lower}" upper="${waist_pan_joint_upper}" velocity="${waist_pan_joint_velocity}" />
    <origin rpy="0 0 0" xyz="0 0 1.152"/>
     <parent link="mid_stomach_link"/>
@@ -144,5 +144,5 @@
   <joint name="waist_roll_joint" type="revolute">
    <axis xyz="1 0 0"/>
-   <limit effort="1000.0" lower="${waist_roll_joint_lower}" upper="${waist_roll_joint_upper}" velocity="${waist_roll_joint_velocity}" />
+   <limit effort="10000.0" lower="${waist_roll_joint_lower}" upper="${waist_roll_joint_upper}" velocity="${waist_roll_joint_velocity}" />
    <origin rpy="0 0 0" xyz="0 0 0.11"/>
     <parent link="top_stomach_link"/>

File: inmoov_description/urdf/config.inertial.urdf.xacro (robot description, xacro)
@@ -7,5 +7,5 @@
   <!-- PLA is 1.25g per 1.0cm^3 -->
   <!-- mass divisor, ros is kilograms-->
-  <xacro:property name="md" value="1000"/>
+  <xacro:property name="md" value="5000"/>
   <!-- inertia divisor, ros is meters, -->
   <!-- assume mass == volume for simplicity -->

File: inmoov_description/urdf/inmoov.gazebo.xacro (robot description, xacro)
@@ -6,7 +6,7 @@
   <xacro:property name="SERVO_MIN" value="-1.5707963267948966"/> <!-- -π/2 -->
   <xacro:property name="SERVO_MAX" value=" 1.5707963267948966"/> <!-- +π/2 -->
-  <xacro:property name="FORCE"     value="200.0"/>                 <!-- Nm-ish; tune -->
+  <xacro:property name="FORCE"     value="1000.0"/>                 <!-- Nm-ish; tune -->
   <!-- Small helper to declare one position-only joint with real torque -->
-  <xacro:macro name="pos_only_joint" params="jname cmd_min:=${SERVO_MIN} cmd_max:=${SERVO_MAX} kp:=60.0 kd:=1.0 ki:=0.0 fmax:=${FORCE}">
+  <xacro:macro name="pos_only_joint" params="jname cmd_min:=${SERVO_MIN} cmd_max:=${SERVO_MAX} kp:=1000.0 kd:=15.0 ki:=0.0 fmax:=${FORCE}">
     <joint name="${jname}">
       <command_interface name="position">
@@ -30,9 +30,16 @@
       <!-- Keep hardware section minimal; per-joint params above actually take effect -->
     </hardware>
+    <!-- Heavier group overrides -->
+    <xacro:pos_only_joint jname="waist_pan_joint"  kp="5200" kd="25" fmax="10000"/>
+    <xacro:pos_only_joint jname="waist_roll_joint" kp="8200" kd="25" fmax="10000"/>
+    <xacro:pos_only_joint jname="r_shoulder_lift_joint" kp="1800" kd="20" fmax="9000"/>
+    <xacro:pos_only_joint jname="r_shoulder_out_joint"  kp="1800" kd="20" fmax="9000"/>
+    <xacro:pos_only_joint jname="r_upper_arm_roll_joint" kp="1600" kd="18" fmax="8000"/>
+    <xacro:pos_only_joint jname="l_shoulder_lift_joint" kp="1800" kd="20" fmax="9000"/>
+    <xacro:pos_only_joint jname="l_shoulder_out_joint"  kp="1800" kd="20" fmax="9000"/>
+    <xacro:pos_only_joint jname="l_upper_arm_roll_joint" kp="1600" kd="18" fmax="8000"/>
     <!-- torso / neck / head -->
-    <xacro:pos_only_joint jname="waist_pan_joint"/>
-    <xacro:pos_only_joint jname="waist_roll_joint"/>
     <xacro:pos_only_joint jname="head_roll_joint"/>
-    <xacro:pos_only_joint jname="head_tilt_joint"/>
+    <xacro:pos_only_joint jname="head_tilt_joint" kp="8200" kd="25" fmax="10000"/>
     <xacro:pos_only_joint jname="head_pan_joint"/>
     <!-- jaw / eyes -->
@@ -41,15 +48,9 @@
     <xacro:pos_only_joint jname="eyes_pan_joint"/>
     <!-- right arm -->
-    <xacro:pos_only_joint jname="r_shoulder_lift_joint"/>
-    <xacro:pos_only_joint jname="r_upper_arm_roll_joint"/>
     <xacro:pos_only_joint jname="r_elbow_flex_joint"/>
-    <xacro:pos_only_joint jname="r_shoulder_out_joint"/>
-    <xacro:pos_only_joint jname="r_wrist_roll_joint" cmd_min="-3.141592653589793" cmd_max="3.141592653589793"/>
+    <xacro:pos_only_joint jname="r_wrist_roll_joint"/>
     <!-- left arm -->
-    <xacro:pos_only_joint jname="l_shoulder_lift_joint"/>
-    <xacro:pos_only_joint jname="l_upper_arm_roll_joint"/>
     <xacro:pos_only_joint jname="l_elbow_flex_joint"/>
-    <xacro:pos_only_joint jname="l_shoulder_out_joint"/>
-    <xacro:pos_only_joint jname="l_wrist_roll_joint" cmd_min="-3.141592653589793" cmd_max="3.141592653589793"/>
+    <xacro:pos_only_joint jname="l_wrist_roll_joint"/>
     <!-- left hand -->
     <xacro:pos_only_joint jname="l_thumb_joint"/>
