Commit message: Now need to fix arms

File: inmoov_description/urdf/config.inertial.urdf.xacro (robot description, xacro)
@@ -7,8 +7,9 @@
   <!-- PLA is 1.25g per 1.0cm^3 -->
   <!-- mass divisor, ros is kilograms-->
-  <xacro:property name="md" value="5000"/>
+  <xacro:property name="rho" value="1000"/>
+  <xacro:property name="md" value="${1e9 / rho}"/>
+  <xacro:property name="id" value="${md * 1e6}"/>
   <!-- inertia divisor, ros is meters, -->
   <!-- assume mass == volume for simplicity -->
-  <xacro:property name="id" value="${ md * md * md}"/>
 <!--
 Opened mesh /home/grey/inmoov_ros/src/inmoov_ros/inmoov_description/meshes/bicep.stl in 6 msec
@@ -33,4 +34,5 @@
   <xacro:macro name="bicep_inertial">
     <inertial>
+      <origin xyz="-0.010079529 0.000072064 -0.081852776" rpy="0 0 0"/>
       <mass value="${281912.656250 / md}"/>
       <inertia
@@ -66,4 +68,5 @@
   <xacro:macro name="bicepcover_inertial">
     <inertial>
+      <origin xyz="0.004113691 0.000023778 -0.098293915" rpy="0 0 0"/>
       <mass value="${176269.609375 / md}"/>
       <inertia
@@ -99,4 +102,5 @@
   <xacro:macro name="camera_inertial">
     <inertial>
+      <origin xyz="0.002337499 -0.000368498 -0.002255082" rpy="0 0 0"/>
       <mass value="${2466.067627 / md}"/>
       <inertia
@@ -132,4 +136,5 @@
   <xacro:macro name="chest_inertial">
     <inertial>
+      <origin xyz="0.016772718 -0.001230909 0.125540794" rpy="0 0 0"/>
       <mass value="${755680.687500 / md}"/>
       <inertia
@@ -165,4 +170,5 @@
   <xacro:macro name="disk_inertial">
     <inertial>
+      <origin xyz="0.020559896 -0.000052606 0.008121016" rpy="0 0 0"/>
       <mass value="${178967.343750 / md}"/>
       <inertia
@@ -198,4 +204,5 @@
   <xacro:macro name="earleftv1_inertial">
     <inertial>
+      <origin xyz="0.003795357 0.007653911 0.002931803" rpy="0 0 0"/>
       <mass value="${ 85197.960938 / md}"/>
       <inertia
@@ -231,4 +238,5 @@
   <xacro:macro name="earrightv1_inertial">
     <inertial>
+      <origin xyz="0.003741870 -0.007651948 0.002376738" rpy="0 0 0"/>
       <mass value="${ 85175.406250 / md}"/>
       <inertia
@@ -264,4 +272,5 @@
   <xacro:macro name="eye_inertial">
     <inertial>
+      <origin xyz="0.003185493 0.000000001 0.000000025" rpy="0 0 0"/>
       <mass value="${ 4659.753906 / md}"/>
       <inertia
@@ -297,4 +306,5 @@
   <xacro:macro name="eyesupport_inertial">
     <inertial>
+      <origin xyz="-0.003586834 -0.000028465 0.001197724" rpy="0 0 0"/>
       <mass value="${ 27550.294922 / md}"/>
       <inertia
@@ -330,4 +340,5 @@
   <xacro:macro name="face_inertial">
     <inertial>
+      <origin xyz="0.019483259 -0.000081941 -0.009738870" rpy="0 0 0"/>
       <mass value="${ 46559.031250 / md}"/>
       <inertia
@@ -363,4 +374,5 @@
   <xacro:macro name="head_inertial">
     <inertial>
+      <origin xyz="0.033712868 -0.000019775 0.019798304" rpy="0 0 0"/>
       <mass value="${ 120499.460938 / md}"/>
       <inertia
@@ -396,4 +408,5 @@
   <xacro:macro name="head_base_inertial">
     <inertial>
+      <origin xyz="0.007293888 0.000021165 0.014839767" rpy="0 0 0"/>
       <mass value="${ 43502.281250 / md}"/>
       <inertia
@@ -429,4 +442,5 @@
   <xacro:macro name="index3_1_inertial">
     <inertial>
+      <origin xyz="0.000327900 -0.000041642 -0.017815184" rpy="0 0 0"/>
       <mass value="${ 4854.550781 / md}"/>
       <inertia
@@ -462,4 +476,5 @@
   <xacro:macro name="index3_2_inertial">
     <inertial>
+      <origin xyz="0.000920736 -0.000011680 -0.010908571" rpy="0 0 0"/>
       <mass value="${ 2911.548828 / md}"/>
       <inertia
@@ -495,4 +510,5 @@
   <xacro:macro name="index3_3_inertial">
     <inertial>
+      <origin xyz="-0.000195631 -0.000042939 -0.012565110" rpy="0 0 0"/>
       <mass value="${ 2754.759033 / md}"/>
       <inertia
@@ -528,4 +544,5 @@
   <xacro:macro name="iris_inertial">
     <inertial>
+      <origin xyz="0.002386165 0.000000047 -0.000099872" rpy="0 0 0"/>
       <mass value="${ 1026.836548 / md}"/>
       <inertia
@@ -561,4 +578,5 @@
   <xacro:macro name="jaw_inertial">
     <inertial>
+      <origin xyz="0.063222282 0.000037192 -0.049244869" rpy="0 0 0"/>
       <mass value="${ 58767.261719 / md}"/>
       <inertia
@@ -594,4 +612,5 @@
   <xacro:macro name="kinectone_inertial">
     <inertial>
+      <origin xyz="0.001100458 0.048963375 0.038179012" rpy="0 0 0"/>
       <mass value="${ 790831.937500 / md}"/>
       <inertia
@@ -627,4 +646,5 @@
   <xacro:macro name="l_cover_hand_inertial">
     <inertial>
+      <origin xyz="0.003708912 0.013324540 0.043250717" rpy="0 0 0"/>
       <mass value="${ 39850.039062 / md}"/>
       <inertia
@@ -660,4 +680,5 @@
   <xacro:macro name="l_cover_handpinky_inertial">
     <inertial>
+      <origin xyz="0.002283108 -0.000345010 0.001597708" rpy="0 0 0"/>
       <mass value="${ 3887.731445 / md}"/>
       <inertia
@@ -693,4 +714,5 @@
   <xacro:macro name="l_cover_handring_inertial">
     <inertial>
+      <origin xyz="0.002592369 0.000223609 -0.001677225" rpy="0 0 0"/>
       <mass value="${ 3507.538086 / md}"/>
       <inertia
@@ -726,4 +748,5 @@
   <xacro:macro name="l_cover_index_inertial">
     <inertial>
+      <origin xyz="0.004354176 -0.000273627 0.000371592" rpy="0 0 0"/>
       <mass value="${ 1635.368652 / md}"/>
       <inertia
@@ -759,4 +782,5 @@
   <xacro:macro name="l_cover_middle_inertial">
     <inertial>
+      <origin xyz="0.004406314 -0.000082271 0.000264647" rpy="0 0 0"/>
       <mass value="${ 1904.471313 / md}"/>
       <inertia
@@ -792,4 +816,5 @@
   <xacro:macro name="l_cover_pinky_inertial">
     <inertial>
+      <origin xyz="0.003877148 -0.000506894 0.001602272" rpy="0 0 0"/>
       <mass value="${ 1285.607300 / md}"/>
       <inertia
@@ -825,4 +850,5 @@
   <xacro:macro name="l_cover_ring_inertial">
     <inertial>
+      <origin xyz="0.004013374 0.000186770 0.001242054" rpy="0 0 0"/>
       <mass value="${ 1466.901733 / md}"/>
       <inertia
@@ -858,4 +884,5 @@
   <xacro:macro name="l_cover_thumb_inertial">
     <inertial>
+      <origin xyz="0.002521784 0.002407381 -0.000141687" rpy="0 0 0"/>
       <mass value="${ 3250.209717 / md}"/>
       <inertia
@@ -891,4 +918,5 @@
   <xacro:macro name="l_eyesupport_inertial">
     <inertial>
+      <origin xyz="-0.004087140 -0.000392808 0.002943427" rpy="0 0 0"/>
       <mass value="${ 11370.105469 / md}"/>
       <inertia
@@ -924,4 +952,5 @@
   <xacro:macro name="l_forearm_inertial">
     <inertial>
+      <origin xyz="-0.006129842 -0.003489157 -0.118607628" rpy="0 0 0"/>
       <mass value="${ 401766.593750 / md}"/>
       <inertia
@@ -957,4 +986,5 @@
   <xacro:macro name="l_hand_inertial">
     <inertial>
+      <origin xyz="-0.000270632 -0.005146427 -0.053579273" rpy="0 0 0"/>
       <mass value="${ 83605.007812 / md}"/>
       <inertia
@@ -990,4 +1020,5 @@
   <xacro:macro name="l_pinky3_1_inertial">
     <inertial>
+      <origin xyz="-0.000456468 0.018407099 -0.005171003" rpy="0 0 0"/>
       <mass value="${ 14892.949219 / md}"/>
       <inertia
@@ -1023,4 +1054,5 @@
   <xacro:macro name="l_ring3_1_inertial">
     <inertial>
+      <origin xyz="-0.000064880 0.015507306 -0.002144598" rpy="0 0 0"/>
       <mass value="${ 10810.309570 / md}"/>
       <inertia
@@ -1056,4 +1088,5 @@
   <xacro:macro name="l_shoulder_inertial">
     <inertial>
+      <origin xyz="-0.001760977 0.046793152 -0.026001684" rpy="0 0 0"/>
       <mass value="${ 322443.343750 / md}"/>
       <inertia
@@ -1089,4 +1122,5 @@
   <xacro:macro name="l_shoulder_base_inertial">
     <inertial>
+      <origin xyz="-0.003377304 -0.011160115 -0.046922394" rpy="0 0 0"/>
       <mass value="${ 266526.968750 / md}"/>
       <inertia
@@ -1122,4 +1156,5 @@
   <xacro:macro name="l_thumb5_1_inertial">
     <inertial>
+      <origin xyz="0.001007494 -0.013727526 -0.002808447" rpy="0 0 0"/>
       <mass value="${ 10044.437500 / md}"/>
       <inertia
@@ -1155,4 +1190,5 @@
   <xacro:macro name="middle3_1_inertial">
     <inertial>
+      <origin xyz="0.000259172 0.000005322 -0.018944950" rpy="0 0 0"/>
       <mass value="${ 5988.140625 / md}"/>
       <inertia
@@ -1188,4 +1224,5 @@
   <xacro:macro name="middle3_2_inertial">
     <inertial>
+      <origin xyz="0.000997151 -0.000059130 -0.011654193" rpy="0 0 0"/>
       <mass value="${ 3588.543701 / md}"/>
       <inertia
@@ -1221,4 +1258,5 @@
   <xacro:macro name="middle3_3_inertial">
     <inertial>
+      <origin xyz="-0.000301118 -0.000030560 -0.013531679" rpy="0 0 0"/>
       <mass value="${ 3395.293457 / md}"/>
       <inertia
@@ -1254,4 +1292,5 @@
   <xacro:macro name="mid_stomach_inertial">
     <inertial>
+      <origin xyz="-0.004659371 -0.000067826 -0.041636871" rpy="0 0 0"/>
       <mass value="${ 1710217.625000 / md}"/>
       <inertia
@@ -1287,4 +1326,5 @@
   <xacro:macro name="pinky3_2_inertial">
     <inertial>
+      <origin xyz="0.000292973 0.000060040 -0.015377484" rpy="0 0 0"/>
       <mass value="${ 3053.924072 / md}"/>
       <inertia
@@ -1320,4 +1360,5 @@
   <xacro:macro name="pinky3_3_inertial">
     <inertial>
+      <origin xyz="0.000831476 -0.000076120 -0.009414209" rpy="0 0 0"/>
       <mass value="${ 1848.707520 / md}"/>
       <inertia
@@ -1353,4 +1394,5 @@
   <xacro:macro name="pinky3_4_inertial">
     <inertial>
+      <origin xyz="-0.000214676 -0.000034577 -0.010846709" rpy="0 0 0"/>
       <mass value="${ 1748.221436 / md}"/>
       <inertia
@@ -1386,4 +1428,5 @@
   <xacro:macro name="r_cover_hand_inertial">
     <inertial>
+      <origin xyz="0.003708912 -0.013324539 0.043250721" rpy="0 0 0"/>
       <mass value="${ 39850.042969 / md}"/>
       <inertia
@@ -1419,4 +1462,5 @@
   <xacro:macro name="r_cover_handpinky_inertial">
     <inertial>
+      <origin xyz="0.002283108 0.000345010 0.001597708" rpy="0 0 0"/>
       <mass value="${ 3887.731445 / md}"/>
       <inertia
@@ -1452,4 +1496,5 @@
   <xacro:macro name="r_cover_handring_inertial">
     <inertial>
+      <origin xyz="0.002592369 -0.000223609 -0.001677225" rpy="0 0 0"/>
       <mass value="${ 3507.538330 / md}"/>
       <inertia
@@ -1485,4 +1530,5 @@
   <xacro:macro name="r_cover_index_inertial">
     <inertial>
+      <origin xyz="0.004354176 0.000273627 0.000371592" rpy="0 0 0"/>
       <mass value="${ 1635.368652 / md}"/>
       <inertia
@@ -1518,4 +1564,5 @@
   <xacro:macro name="r_cover_middle_inertial">
     <inertial>
+      <origin xyz="0.004406314 0.000082271 0.000264647" rpy="0 0 0"/>
       <mass value="${ 1904.471313 / md}"/>
       <inertia
@@ -1551,4 +1598,5 @@
   <xacro:macro name="r_cover_pinky_inertial">
     <inertial>
+      <origin xyz="0.003877148 0.000506894 0.001602272" rpy="0 0 0"/>
       <mass value="${ 1285.607300 / md}"/>
       <inertia
@@ -1584,4 +1632,5 @@
   <xacro:macro name="r_cover_ring_inertial">
     <inertial>
+      <origin xyz="0.004013374 -0.000186770 0.001242054" rpy="0 0 0"/>
       <mass value="${ 1466.901733 / md}"/>
       <inertia
@@ -1617,4 +1666,5 @@
   <xacro:macro name="r_cover_thumb_inertial">
     <inertial>
+      <origin xyz="0.002521784 -0.002407381 -0.000141687" rpy="0 0 0"/>
       <mass value="${ 3250.209961 / md}"/>
       <inertia
@@ -1650,4 +1700,5 @@
   <xacro:macro name="r_eyesupport_inertial">
     <inertial>
+      <origin xyz="-0.004087140 0.000392808 0.002943427" rpy="0 0 0"/>
       <mass value="${ 11370.105469 / md}"/>
       <inertia
@@ -1683,4 +1734,5 @@
   <xacro:macro name="r_forearm_inertial">
     <inertial>
+      <origin xyz="-0.006129843 0.003489157 -0.118607635" rpy="0 0 0"/>
       <mass value="${ 401766.593750 / md}"/>
       <inertia
@@ -1716,4 +1768,5 @@
   <xacro:macro name="r_hand_inertial">
     <inertial>
+      <origin xyz="-0.000270633 0.005146428 -0.053579273" rpy="0 0 0"/>
       <mass value="${ 83605.000000 / md}"/>
       <inertia
@@ -1749,4 +1802,5 @@
   <xacro:macro name="ring3_2_inertial">
     <inertial>
+      <origin xyz="0.000230179 -0.000040497 -0.016867937" rpy="0 0 0"/>
       <mass value="${ 4222.559082 / md}"/>
       <inertia
@@ -1782,4 +1836,5 @@
   <xacro:macro name="ring3_3_inertial">
     <inertial>
+      <origin xyz="0.000920449 -0.000022269 -0.010337892" rpy="0 0 0"/>
       <mass value="${ 2530.003662 / md}"/>
       <inertia
@@ -1815,4 +1870,5 @@
   <xacro:macro name="ring3_4_inertial">
     <inertial>
+      <origin xyz="-0.000248927 0.000051272 -0.012062567" rpy="0 0 0"/>
       <mass value="${ 2393.758301 / md}"/>
       <inertia
@@ -1848,4 +1904,5 @@
   <xacro:macro name="r_pinky3_1_inertial">
     <inertial>
+      <origin xyz="-0.000456468 -0.018407099 -0.005171003" rpy="0 0 0"/>
       <mass value="${ 14892.949219 / md}"/>
       <inertia
@@ -1881,4 +1938,5 @@
   <xacro:macro name="r_ring3_1_inertial">
     <inertial>
+      <origin xyz="-0.000064880 -0.015507305 -0.002144598" rpy="0 0 0"/>
       <mass value="${ 10810.309570 / md}"/>
       <inertia
@@ -1914,4 +1972,5 @@
   <xacro:macro name="r_shoulder_inertial">
     <inertial>
+      <origin xyz="-0.001760979 -0.046793152 -0.026001682" rpy="0 0 0"/>
       <mass value="${ 322443.343750 / md}"/>
       <inertia
@@ -1947,4 +2006,5 @@
   <xacro:macro name="r_shoulder_base_inertial">
     <inertial>
+      <origin xyz="-0.003377304 0.011160116 -0.046922394" rpy="0 0 0"/>
       <mass value="${ 266526.968750 / md}"/>
       <inertia
@@ -1980,4 +2040,5 @@
   <xacro:macro name="r_thumb5_1_inertial">
     <inertial>
+      <origin xyz="0.001007495 0.013727525 -0.002808447" rpy="0 0 0"/>
       <mass value="${ 10044.436523 / md}"/>
       <inertia
@@ -2013,4 +2074,5 @@
   <xacro:macro name="skull_inertial">
     <inertial>
+      <origin xyz="-0.003423218 0.001018229 0.101525459" rpy="0 0 0"/>
       <mass value="${ 422313.062500 / md}"/>
       <inertia
@@ -2046,4 +2108,5 @@
   <xacro:macro name="thumb5_2_inertial">
     <inertial>
+      <origin xyz="-0.000025869 -0.000050593 -0.016259710" rpy="0 0 0"/>
       <mass value="${ 7511.052246 / md}"/>
       <inertia
@@ -2079,4 +2142,5 @@
   <xacro:macro name="thumb5_3_inertial">
     <inertial>
+      <origin xyz="0.000392466 -0.000002426 -0.013323187" rpy="0 0 0"/>
       <mass value="${ 5812.545410 / md}"/>
       <inertia
@@ -2112,4 +2176,5 @@
   <xacro:macro name="top_stomach_inertial">
     <inertial>
+      <origin xyz="-0.003812517 -0.000053483 0.044282845" rpy="0 0 0"/>
       <mass value="${ 1144889.750000 / md}"/>
       <inertia
@@ -2145,4 +2210,5 @@
   <xacro:macro name="torso_inertial">
     <inertial>
+      <origin xyz="-0.003839768 -0.000257000 0.172243729" rpy="0 0 0"/>
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
File: inmoov_description/urdf/inmoov.gazebo.xacro (robot description, xacro)
@@ -8,5 +8,5 @@
   <xacro:property name="FORCE"     value="1000.0"/>                 <!-- Nm-ish; tune -->
   <!-- Small helper to declare one position-only joint with real torque -->
-  <xacro:macro name="pos_only_joint" params="jname cmd_min:=${SERVO_MIN} cmd_max:=${SERVO_MAX} kp:=1000.0 kd:=15.0 ki:=0.0 fmax:=${FORCE}">
+  <xacro:macro name="pos_only_joint" params="jname cmd_min:=${SERVO_MIN} cmd_max:=${SERVO_MAX} kp:=60.0 kd:=1.0 ki:=0.0 fmax:=${FORCE}">
     <joint name="${jname}">
       <command_interface name="position">
@@ -31,15 +31,15 @@
     </hardware>
     <!-- Heavier group overrides -->
-    <xacro:pos_only_joint jname="waist_pan_joint"  kp="5200" kd="25" fmax="10000"/>
-    <xacro:pos_only_joint jname="waist_roll_joint" kp="8200" kd="25" fmax="10000"/>
-    <xacro:pos_only_joint jname="r_shoulder_lift_joint" kp="1800" kd="20" fmax="9000"/>
-    <xacro:pos_only_joint jname="r_shoulder_out_joint"  kp="1800" kd="20" fmax="9000"/>
-    <xacro:pos_only_joint jname="r_upper_arm_roll_joint" kp="1600" kd="18" fmax="8000"/>
-    <xacro:pos_only_joint jname="l_shoulder_lift_joint" kp="1800" kd="20" fmax="9000"/>
-    <xacro:pos_only_joint jname="l_shoulder_out_joint"  kp="1800" kd="20" fmax="9000"/>
-    <xacro:pos_only_joint jname="l_upper_arm_roll_joint" kp="1600" kd="18" fmax="8000"/>
+    <xacro:pos_only_joint jname="waist_pan_joint"  kp="100" kd="5" fmax="2000"/>
+    <xacro:pos_only_joint jname="waist_roll_joint" kp="100" kd="5" fmax="2000"/>
+    <xacro:pos_only_joint jname="r_shoulder_lift_joint" kp="100" kd="5" fmax="2000"/>
+    <xacro:pos_only_joint jname="r_shoulder_out_joint"  kp="100" kd="5" fmax="2000"/>
+    <xacro:pos_only_joint jname="r_upper_arm_roll_joint" kp="100" kd="5" fmax="2000"/>
+    <xacro:pos_only_joint jname="l_shoulder_lift_joint" kp="100" kd="5" fmax="2000"/>
+    <xacro:pos_only_joint jname="l_shoulder_out_joint"  kp="100" kd="5" fmax="2000"/>
+    <xacro:pos_only_joint jname="l_upper_arm_roll_joint" kp="100" kd="5" fmax="2000"/>
     <!-- torso / neck / head -->
-    <xacro:pos_only_joint jname="head_roll_joint"/>
-    <xacro:pos_only_joint jname="head_tilt_joint" kp="8200" kd="25" fmax="10000"/>
+    <xacro:pos_only_joint jname="head_roll_joint" />
+    <xacro:pos_only_joint jname="head_tilt_joint" kp="100" kd="5" fmax="2000"/>
     <xacro:pos_only_joint jname="head_pan_joint"/>
     <!-- jaw / eyes -->
@@ -49,5 +49,5 @@
     <!-- right arm -->
     <xacro:pos_only_joint jname="r_elbow_flex_joint"/>
-    <xacro:pos_only_joint jname="r_wrist_roll_joint"/>
+    <xacro:pos_only_joint jname="r_wrist_roll_joint" />
     <!-- left arm -->
     <xacro:pos_only_joint jname="l_elbow_flex_joint"/>
