Commit message: Add ros2_control hardware driver so RViz moves the real InMoov
Three-package split (description / hardware / bringup):

* inmoov_hardware (new) - a hardware_interface::SystemInterface that turns
  URDF joint positions into MyRobotLab servo commands. Runs entirely on the
  ROS2 machine and speaks to MRL's plain-HTTP Nixie API on
  pi5-inmoov.local:8888; nothing is installed on the pi5.

* inmoov_bringup (new) - controller config + the two launch paths:
  inmoov_real.launch.py (ros2_control) and inmoov_sliders.launch.py
  (joint_state_publisher_gui -> /joint_states -> relay). Both share one
  mapping implementation, libinmoov_mapping.

* inmoov_description - gains an argument-gated <ros2_control> macro.
  use_real_hardware:=true selects the real driver and drops Gazebo entirely;
  the default is unchanged, and the package still has no dependency on
  inmoov_hardware. display.launch.py and gazebo.launch.py are untouched.

The mapping (config/inmoov_joint_map.yaml) anchors every joint at a home
radian value that maps exactly onto the servo's REST position, then scales
each side independently onto the servo's real [min,max]. servo min/max/rest
were read LIVE from MRL, not taken from the static servo_map.py table, and
are re-read on activation. 28 of the 53 URDF joints have a servo; the rest
(finger sub-links, second eye pan) are marked disabled and ignored cleanly.

Safety: output is clamped to the servo range and then to an optional safety
cap; enabled_groups gates which body parts are driven at all and defaults to
head only; dry_run logs every intended move and sends nothing. Held poses are
re-asserted every 0.5s because InMoov servos droop.

read() reports the last commanded position - MRL has no real feedback and the
code says so rather than pretending otherwise.

Tested: clean colcon build, 19 offline arithmetic tests green, both launch
paths proven end-to-end in dry-run. Live on the robot: head_pan_joint only,
0 -> +0.2 -> 0 -> -0.2 -> 0 rad capped to +/-8 deg, MRL reported rothead
90 -> 97 -> 90 -> 83 -> 90 and rested on shutdown. Arms, hands and torso are
wired but have never been commanded, and no direction sign has been confirmed
by eye - see "What is unverified" in inmoov_hardware/README.md.

Co-Authored-By: Claude Opus 5 (1M context) <noreply@anthropic.com>
Claude-Session: https://claude.ai/code/session_01Kpk5vJ7u2Qct1dnDk8Kg4X

File: inmoov_description/robots/inmoov.urdf.xacro (robot description, xacro)
@@ -11,5 +11,34 @@
 <xacro:include filename="$(find inmoov_description)/urdf/asmArm.urdf.xacro" />
 <xacro:include filename="$(find inmoov_description)/urdf/asmHand.urdf.xacro" />
+<!-- ==========================================================================
+     Control back-end selection.
+     use_real_hardware:=false (default) -> Gazebo Sim ros2_control, exactly as before.
+     use_real_hardware:=true            -> the inmoov_hardware SystemInterface that drives
+                                           the physical robot through MyRobotLab, and NO
+                                           Gazebo plugin at all (there is nothing to
+                                           simulate when the real robot is the plant).
+     Both files only DEFINE macros, so including them unconditionally is free; only the
+     invocation below is gated. inmoov_description gains no dependency on inmoov_hardware
+     from this — the plugin is a string that pluginlib resolves at run time.
+     ========================================================================== -->
+<xacro:arg name="use_real_hardware" default="false"/>
+<xacro:arg name="mrl_host"          default="pi5-inmoov.local"/>
+<xacro:arg name="mrl_port"          default="8888"/>
+<xacro:arg name="enabled_groups"    default="head"/>
+<xacro:arg name="dry_run"           default="false"/>
+<xacro:arg name="joint_map"         default=""/>
 <xacro:include filename="$(find inmoov_description)/urdf/inmoov.gazebo.xacro" />
+<xacro:include filename="$(find inmoov_description)/urdf/inmoov.ros2_control.xacro" />
+<xacro:if value="$(arg use_real_hardware)">
+  <xacro:inmoov_real_ros2_control
+      mrl_host="$(arg mrl_host)"
+      mrl_port="$(arg mrl_port)"
+      enabled_groups="$(arg enabled_groups)"
+      dry_run="$(arg dry_run)"
+      joint_map="$(arg joint_map)"/>
+</xacro:if>
+<xacro:unless value="$(arg use_real_hardware)">
+  <xacro:inmoov_gazebo_control/>
+</xacro:unless>
   <link name="world"/>
     <xacro:virtual_inertial/>

File: inmoov_description/urdf/inmoov.gazebo.xacro (robot description, xacro)
@@ -22,55 +22,60 @@
     </joint>
   </xacro:macro>
-  <!-- ============================================================
-       ros2_control for Gazebo Sim (position-only on all joints)
-       ============================================================ -->
-  <ros2_control name="inmoov_system" type="system">
-    <hardware>
-      <plugin>gz_ros2_control/GazeboSimSystem</plugin>
-      <!-- Keep hardware section minimal; per-joint params above actually take effect -->
-    </hardware>
-    <!-- Heavier group overrides -->
-    <xacro:pos_only_joint jname="waist_pan_joint"  kp="100" kd="5" fmax="2000"/>
-    <xacro:pos_only_joint jname="waist_roll_joint" kp="100" kd="5" fmax="2000"/>
-    <xacro:pos_only_joint jname="r_shoulder_lift_joint" kp="100" kd="5" fmax="2000"/>
-    <xacro:pos_only_joint jname="r_shoulder_out_joint"  kp="100" kd="5" fmax="2000"/>
-    <xacro:pos_only_joint jname="r_upper_arm_roll_joint" kp="100" kd="5" fmax="2000"/>
-    <xacro:pos_only_joint jname="l_shoulder_lift_joint" kp="100" kd="5" fmax="2000"/>
-    <xacro:pos_only_joint jname="l_shoulder_out_joint"  kp="100" kd="5" fmax="2000"/>
-    <xacro:pos_only_joint jname="l_upper_arm_roll_joint" kp="100" kd="5" fmax="2000"/>
-    <!-- torso / neck / head -->
-    <xacro:pos_only_joint jname="head_roll_joint" />
-    <xacro:pos_only_joint jname="head_tilt_joint" kp="100" kd="5" fmax="2000"/>
-    <xacro:pos_only_joint jname="head_pan_joint"/>
-    <!-- jaw / eyes -->
-    <xacro:pos_only_joint jname="jaw_joint"/>
-    <xacro:pos_only_joint jname="eyes_tilt_joint"/>
-    <xacro:pos_only_joint jname="eyes_pan_joint"/>
-    <!-- right arm -->
-    <xacro:pos_only_joint jname="r_elbow_flex_joint"/>
-    <xacro:pos_only_joint jname="r_wrist_roll_joint" />
-    <!-- left arm -->
-    <xacro:pos_only_joint jname="l_elbow_flex_joint"/>
-    <xacro:pos_only_joint jname="l_wrist_roll_joint"/>
-    <!-- left hand -->
-    <xacro:pos_only_joint jname="l_thumb_joint"/>
-    <xacro:pos_only_joint jname="l_index_joint"/>
-    <xacro:pos_only_joint jname="l_middle_joint"/>
-    <xacro:pos_only_joint jname="l_ring_joint"/>
-    <xacro:pos_only_joint jname="l_pinky_joint"/>
-    <!-- right hand -->
-    <xacro:pos_only_joint jname="r_thumb_joint"/>
-    <xacro:pos_only_joint jname="r_index_joint"/>
-    <xacro:pos_only_joint jname="r_middle_joint"/>
-    <xacro:pos_only_joint jname="r_ring_joint"/>
-    <xacro:pos_only_joint jname="r_pinky_joint"/>
-  </ros2_control>
-  <!-- Gazebo Sim system plugin loader -->
-  <gazebo>
-    <plugin filename="libgz_ros2_control-system.so"
-            name="gz_ros2_control::GazeboSimROS2ControlPlugin">
-      <parameters>$(find inmoov_description)/config/controllers.yaml</parameters>
-    </plugin>
-  </gazebo>
+  <!-- Everything that follows is SIMULATION-ONLY and is now wrapped in a macro so the
+       top-level robot xacro can leave it out entirely when driving real hardware.
+       Invoke with <xacro:inmoov_gazebo_control/>. -->
+  <xacro:macro name="inmoov_gazebo_control">
+    <!-- ============================================================
+         ros2_control for Gazebo Sim (position-only on all joints)
+         ============================================================ -->
+    <ros2_control name="inmoov_system" type="system">
+      <hardware>
+        <plugin>gz_ros2_control/GazeboSimSystem</plugin>
+        <!-- Keep hardware section minimal; per-joint params above actually take effect -->
+      </hardware>
+      <!-- Heavier group overrides -->
+      <xacro:pos_only_joint jname="waist_pan_joint"  kp="100" kd="5" fmax="2000"/>
+      <xacro:pos_only_joint jname="waist_roll_joint" kp="100" kd="5" fmax="2000"/>
+      <xacro:pos_only_joint jname="r_shoulder_lift_joint" kp="100" kd="5" fmax="2000"/>
+      <xacro:pos_only_joint jname="r_shoulder_out_joint"  kp="100" kd="5" fmax="2000"/>
+      <xacro:pos_only_joint jname="r_upper_arm_roll_joint" kp="100" kd="5" fmax="2000"/>
+      <xacro:pos_only_joint jname="l_shoulder_lift_joint" kp="100" kd="5" fmax="2000"/>
+      <xacro:pos_only_joint jname="l_shoulder_out_joint"  kp="100" kd="5" fmax="2000"/>
+      <xacro:pos_only_joint jname="l_upper_arm_roll_joint" kp="100" kd="5" fmax="2000"/>
+      <!-- torso / neck / head -->
+      <xacro:pos_only_joint jname="head_roll_joint" />
+      <xacro:pos_only_joint jname="head_tilt_joint" kp="100" kd="5" fmax="2000"/>
+      <xacro:pos_only_joint jname="head_pan_joint"/>
+      <!-- jaw / eyes -->
+      <xacro:pos_only_joint jname="jaw_joint"/>
+      <xacro:pos_only_joint jname="eyes_tilt_joint"/>
+      <xacro:pos_only_joint jname="eyes_pan_joint"/>
+      <!-- right arm -->
+      <xacro:pos_only_joint jname="r_elbow_flex_joint"/>
+      <xacro:pos_only_joint jname="r_wrist_roll_joint" />
+      <!-- left arm -->
+      <xacro:pos_only_joint jname="l_elbow_flex_joint"/>
+      <xacro:pos_only_joint jname="l_wrist_roll_joint"/>
+      <!-- left hand -->
+      <xacro:pos_only_joint jname="l_thumb_joint"/>
+      <xacro:pos_only_joint jname="l_index_joint"/>
+      <xacro:pos_only_joint jname="l_middle_joint"/>
+      <xacro:pos_only_joint jname="l_ring_joint"/>
+      <xacro:pos_only_joint jname="l_pinky_joint"/>
+      <!-- right hand -->
+      <xacro:pos_only_joint jname="r_thumb_joint"/>
+      <xacro:pos_only_joint jname="r_index_joint"/>
+      <xacro:pos_only_joint jname="r_middle_joint"/>
+      <xacro:pos_only_joint jname="r_ring_joint"/>
+      <xacro:pos_only_joint jname="r_pinky_joint"/>
+    </ros2_control>
+    <!-- Gazebo Sim system plugin loader -->
+    <gazebo>
+      <plugin filename="libgz_ros2_control-system.so"
+              name="gz_ros2_control::GazeboSimROS2ControlPlugin">
+        <parameters>$(find inmoov_description)/config/controllers.yaml</parameters>
+      </plugin>
+    </gazebo>
+  </xacro:macro>
   <!-- (colors etc below this line are fine to keep as you had) -->
 </robot>

Commit message: Simple launch files, and fix the joint sign conventions in the MODEL
Two separate jobs, both driven by driving the thing.

LAUNCH FILES. Four files, one job each, replacing two whose names were backwards
(inmoov_real was the CONTROLLER path; inmoov_sliders was the one that actually drove the
real robot, which is most of why the README read badly):

    real.launch.py        RViz + sliders + the real robot          <- the one you want
    sim.launch.py         Gazebo + RViz + sliders
    view.launch.py        model only, nothing connected
    controller.launch.py  the real robot via ros2_control

dry_run is an argument on the two that touch hardware, not a mode to remember. A mode:=
switch on one file was tried first and thrown away: one wrong word and you are driving a
robot you meant to simulate.

controller.launch.py keeps the sliders working, which it could not before. There
/joint_states belongs to joint_state_broadcaster -- the robot reporting where it IS -- so
the sliders are remapped to slider_joint_states and a new bridge node forwards them to the
controller's command topic. NOTE: that bridge has never had a message through it.

README rewritten to lead with the five commands, then the one-driver-at-a-time rule, then
why the servos are deliberately not held.

SIGN CONVENTIONS, fixed in the MODEL not the driver. Fixing them with the driver's invert
flag would have made the simulator and the real robot disagree, which is worse than the bug.

  shoulder_out, wrist_roll: the same slider value moved one arm up and the other down.
    config.yaml states the right side's goals as negatives, so both sides shared an axis
    while their ranges ran opposite ways. Right axis negated AND limits negated: identical
    physical motion, symmetric numbering.

  shoulder_lift: positive moved the arms BACKWARD. 135 degrees of the travel lived on the
    negative side, so the useful direction meant dragging down. Negated on both sides (the
    axis is in the shared ${side} macro, so one edit does both).

  wrist_roll again: ran [0, 3.142] with rest at 1.571, and the GUI starts a slider at zero
    when zero is in range -- so the wrists began fully rotated one way. Re-centred on zero
    at [-1.571, 1.571], same travel, slider centre now IS the rest position.

Every joint whose convention changed had its map entry follow (limits, home, invert) and is
back to `verified: none`. Nine directions were confirmed by eye today; these are not among
them.

A geometric check of all 22 left/right pairs is what found shoulder_out and wrist_roll --
comparing raw <axis> is not enough because the parent frames differ, so it walks the chain
into world coordinates and applies the mirror condition a_R == -M a_L. It still reports
upper_arm_roll and three finger sub-links as unmirrored: upper_arm_roll is left alone
pending a decision, and the fingers are geometry-only links with one tendon servo behind
them which Simon confirmed work correctly on the robot. Reality beats the checker.

Also: the KnownHeadPanNumbers test encoded the pre-flip direction and now asserts the
mirrored values, plus EXPECT_TRUE(invert) so a direction confirmed by eye cannot be
silently unset. And the ros2_control xacro still defaulted hold_refresh_s to 0.5, silently
overriding the C++ default of 0 -- so the controller path was still pulsing the servos
after this morning's change. Only the relay path had actually stopped.

Co-Authored-By: Claude Opus 5 (1M context) <noreply@anthropic.com>
Claude-Session: https://claude.ai/code/session_01Kpk5vJ7u2Qct1dnDk8Kg4X

File: inmoov_description/robots/inmoov.urdf.xacro (robot description, xacro)
@@ -128,5 +128,5 @@
   <xacro:arm side="r" flip="1" covers="yes" />
   <joint name="r_shoulder_out_joint" type="revolute">
-   <axis xyz="1 0 0"/>
+   <axis xyz="-1 0 0"/>
    <limit effort="10000.0" lower="${r_shoulder_out_joint_lower}" upper="${r_shoulder_out_joint_upper}" velocity="${r_shoulder_out_joint_velocity}" />
    <origin rpy="0 0 0" xyz="0 -0.143 0.298"/>
@@ -136,5 +136,5 @@
   <xacro:hand side="r" flip="1" covers="yes" />
   <joint name="r_wrist_roll_joint" type="revolute">
-   <axis xyz="0 0 1"/>
+   <axis xyz="0 0 -1"/>
    <limit effort="10000.0" lower="${r_wrist_roll_joint_lower}" upper="${r_wrist_roll_joint_upper}" velocity="${r_wrist_roll_joint_velocity}" />
    <origin rpy="0 0 0" xyz="-0.0144 0.01  -0.2885"/>

File: inmoov_description/urdf/asmArm.urdf.xacro (robot description, xacro)
@@ -98,5 +98,5 @@
 </link>
   <joint name="${side}_shoulder_lift_joint" type="revolute">
-    <axis xyz="0 1 0"/>
+    <axis xyz="0 -1 0"/>
     <xacro:if value="${side == 'l'}">
       <limit effort="10000.0" lower="${l_shoulder_lift_joint_lower}" upper="${l_shoulder_lift_joint_upper}" velocity="${l_shoulder_lift_joint_velocity}" />

File: inmoov_description/urdf/config.joints.urdf.xacro (robot description, xacro)
@@ -8,6 +8,6 @@
   <xacro:property name="r_middle_joint_upper"            value="${r*c['joints']['r_middle_joint']['maxGoal']}" />
   <xacro:property name="r_middle_joint_velocity"         value="${r*c['joints']['r_middle_joint']['maxSpeed']}" />
-  <xacro:property name="r_shoulder_lift_joint_lower"     value="${r*c['joints']['r_shoulder_lift_joint']['maxGoal']}" />
-  <xacro:property name="r_shoulder_lift_joint_upper"     value="${r*c['joints']['r_shoulder_lift_joint']['minGoal']}" />
+  <xacro:property name="r_shoulder_lift_joint_lower"     value="${-r*c['joints']['r_shoulder_lift_joint']['minGoal']}" />
+  <xacro:property name="r_shoulder_lift_joint_upper"     value="${-r*c['joints']['r_shoulder_lift_joint']['maxGoal']}" />
   <xacro:property name="r_shoulder_lift_joint_velocity"  value="${r*c['joints']['r_shoulder_lift_joint']['maxSpeed']}" />
   <xacro:property name="l_ring_joint_lower"              value="${r*c['joints']['l_ring_joint']['minGoal']}" />
@@ -23,6 +23,6 @@
   <xacro:property name="waist_roll_joint_upper"          value="${r*c['joints']['waist_roll_joint']['minGoal']}" />
   <xacro:property name="waist_roll_joint_velocity"       value="${r*c['joints']['waist_roll_joint']['maxSpeed']}" />
-  <xacro:property name="r_wrist_roll_joint_lower"        value="${r*c['joints']['r_wrist_roll_joint']['maxGoal']}" />
-  <xacro:property name="r_wrist_roll_joint_upper"        value="${r*c['joints']['r_wrist_roll_joint']['minGoal']}" />
+  <xacro:property name="r_wrist_roll_joint_lower"        value="${r*(c['joints']['r_wrist_roll_joint']['maxGoal'] - c['joints']['r_wrist_roll_joint']['minGoal'])/2}" />
+  <xacro:property name="r_wrist_roll_joint_upper"        value="${-(r*(c['joints']['r_wrist_roll_joint']['maxGoal'] - c['joints']['r_wrist_roll_joint']['minGoal'])/2)}" />
   <xacro:property name="r_wrist_roll_joint_velocity"     value="${r*c['joints']['r_wrist_roll_joint']['maxSpeed']}" />
   <xacro:property name="l_middle_joint_lower"            value="${r*c['joints']['l_middle_joint']['minGoal']}" />
@@ -38,6 +38,6 @@
   <xacro:property name="jaw_joint_upper"                 value="${r*c['joints']['jaw_joint']['maxGoal']}" />
   <xacro:property name="jaw_joint_velocity"              value="${r*c['joints']['jaw_joint']['maxSpeed']}" />
-  <xacro:property name="l_wrist_roll_joint_lower"        value="${r*c['joints']['l_wrist_roll_joint']['maxGoal']}" />
-  <xacro:property name="l_wrist_roll_joint_upper"        value="${r*c['joints']['l_wrist_roll_joint']['minGoal']}" />
+  <xacro:property name="l_wrist_roll_joint_lower"        value="${r*(c['joints']['l_wrist_roll_joint']['maxGoal'] - c['joints']['l_wrist_roll_joint']['minGoal'])/2}" />
+  <xacro:property name="l_wrist_roll_joint_upper"        value="${-(r*(c['joints']['l_wrist_roll_joint']['maxGoal'] - c['joints']['l_wrist_roll_joint']['minGoal'])/2)}" />
   <xacro:property name="l_wrist_roll_joint_velocity"     value="${r*c['joints']['l_wrist_roll_joint']['maxSpeed']}" />
   <xacro:property name="r_elbow_flex_joint_lower"        value="${r*c['joints']['r_elbow_flex_joint']['maxGoal']}" />
@@ -50,6 +50,6 @@
   <xacro:property name="r_ring_joint_upper"              value="${r*c['joints']['r_ring_joint']['maxGoal']}" />
   <xacro:property name="r_ring_joint_velocity"           value="${r*c['joints']['r_ring_joint']['maxSpeed']}" />
-  <xacro:property name="l_shoulder_lift_joint_lower"     value="${r*c['joints']['l_shoulder_lift_joint']['maxGoal']}" />
-  <xacro:property name="l_shoulder_lift_joint_upper"     value="${r*c['joints']['l_shoulder_lift_joint']['minGoal']}" />
+  <xacro:property name="l_shoulder_lift_joint_lower"     value="${-r*c['joints']['l_shoulder_lift_joint']['minGoal']}" />
+  <xacro:property name="l_shoulder_lift_joint_upper"     value="${-r*c['joints']['l_shoulder_lift_joint']['maxGoal']}" />
   <xacro:property name="l_shoulder_lift_joint_velocity"  value="${r*c['joints']['l_shoulder_lift_joint']['maxSpeed']}" />
   <xacro:property name="eyes_tilt_joint_lower"           value="${r*c['joints']['eyes_tilt_joint']['maxGoal']}" />
@@ -86,6 +86,6 @@
   <xacro:property name="head_tilt_joint_upper"           value="${r*c['joints']['head_tilt_joint']['maxGoal']}" />
   <xacro:property name="head_tilt_joint_velocity"        value="${r*c['joints']['head_tilt_joint']['maxSpeed']}" />
-  <xacro:property name="r_shoulder_out_joint_lower"      value="${r*c['joints']['r_shoulder_out_joint']['maxGoal']}" />
-  <xacro:property name="r_shoulder_out_joint_upper"      value="${r*c['joints']['r_shoulder_out_joint']['minGoal']}" />
+  <xacro:property name="r_shoulder_out_joint_lower"      value="${-r*c['joints']['r_shoulder_out_joint']['minGoal']}" />
+  <xacro:property name="r_shoulder_out_joint_upper"      value="${-r*c['joints']['r_shoulder_out_joint']['maxGoal']}" />
   <xacro:property name="r_shoulder_out_joint_velocity"   value="${r*c['joints']['r_shoulder_out_joint']['maxSpeed']}" />
 </robot>

File: inmoov_description/urdf/inmoov.ros2_control.xacro (robot description, xacro)
@@ -19,5 +19,5 @@
                        joint_map:=''
                        refresh_limits:='true'
-                       hold_refresh_s:=0.5
+                       hold_refresh_s:=0.0
                        move_epsilon_deg:=1.0
                        require_mrl:='true'">
